File: hexahub.kicad_pcb (KiCad board)
At the start: 2 copper layers, 21 parts, among them J1 USB_C_Receptacle, J3 U235-091N-4BLRC16-2, J4 USB3_A, U1 TPS62932DRLR, U10 TPD4E02B04, U11 AP7313-12SAG-7, U12 TPD4E02B04, U14 TPD4E02B04, U15 ESD122, U2 TPD4E02B04, U3 HD3SS3212, U4 TPD4E02B04, U5 TPS65987DDH, U6 ACT5101, U7 ATtiny3227-M, U8 USB5807C, U9 ESD122

Commit message: layout
Parts:
- removed J1: USB_C_Receptacle, Connector_USB:USB_C_Receptacle_Molex-1054500101
- removed J4: USB3_A, Connector_USB:USB3_A_Receptacle_Wuerth_692122030100
- added C10: 10u, Capacitor_SMD:C_0402_1005Metric, F.Cu at (0.95, 18.4)
- added C100: 100u, Capacitor_SMD:CP_Elec_8x10.5, F.Cu at (50.9, 14.6)
- added C101: 1u, Capacitor_SMD:C_0402_1005Metric, F.Cu at (59.0, 21.1)
- added C102: 100n, Capacitor_SMD:C_0402_1005Metric, F.Cu at (59.0, 23.1)
- added C103: 100n, Capacitor_SMD:C_0402_1005Metric, F.Cu at (59.0, 25.1)
- added C104: 100n, Capacitor_SMD:C_0402_1005Metric, F.Cu at (59.0, 27.0)
- added C105: 220p, Capacitor_SMD:C_0402_1005Metric, F.Cu at (59.0, 29.0)
- added C106: 220p, Capacitor_SMD:C_0402_1005Metric, F.Cu at (59.0, 31.0)
- added C107: 1u, Capacitor_SMD:C_0402_1005Metric, F.Cu at (61.9, 17.1)
- added C108: 1n, Capacitor_SMD:C_0402_1005Metric, F.Cu at (61.9, 19.1)
- added C109: DNP, Capacitor_SMD:C_0402_1005Metric, F.Cu at (61.9, 21.1)
- added C11: 100n, Capacitor_SMD:C_0402_1005Metric, F.Cu at (0.95, 20.4)
- added C110: DNP, Capacitor_SMD:C_0402_1005Metric, F.Cu at (61.9, 23.1)
- added C111: 100n, Capacitor_SMD:C_0402_1005Metric, F.Cu at (61.9, 25.1)
- added C112: 100p, Capacitor_SMD:C_0402_1005Metric, F.Cu at (61.9, 27.0)
- added C113: 100n, Capacitor_SMD:C_0402_1005Metric, F.Cu at (61.9, 29.0)
- added C114: 100n, Capacitor_SMD:C_0402_1005Metric, F.Cu at (61.9, 31.0)
- added C115: 100n, Capacitor_SMD:C_0402_1005Metric, F.Cu at (64.8, 17.1)
- added C116: 100n, Capacitor_SMD:C_0402_1005Metric, F.Cu at (64.8, 19.1)
- added C117: 100n, Capacitor_SMD:C_0402_1005Metric, F.Cu at (64.8, 21.1)
- added C118: 100n, Capacitor_SMD:C_0402_1005Metric, F.Cu at (64.8, 23.1)
- added C119: 100n, Capacitor_SMD:C_0402_1005Metric, F.Cu at (64.8, 25.1)
- added C12: 100n, Capacitor_SMD:C_0402_1005Metric, F.Cu at (0.95, 22.4)
- added C120: 47n, Capacitor_SMD:C_0402_1005Metric, F.Cu at (14.3, 61.2)
- added C121: 47n, Capacitor_SMD:C_0402_1005Metric, F.Cu at (14.3, 63.2)
- added C122: 100u, Capacitor_SMD:CP_Elec_8x10.5, F.Cu at (6.17, 48.7)
- added C123: 100u, Capacitor_SMD:CP_Elec_8x10.5, F.Cu at (6.17, 58.7)
- added C124: 1u, Capacitor_SMD:C_0402_1005Metric, F.Cu at (14.3, 65.2)
- added C125: 100n, Capacitor_SMD:C_0402_1005Metric, F.Cu at (14.3, 67.2)
- added C126: 100n, Capacitor_SMD:C_0402_1005Metric, F.Cu at (14.3, 69.2)
- added C127: 100n, Capacitor_SMD:C_0402_1005Metric, F.Cu at (14.3, 71.2)
- added C128: 220p, Capacitor_SMD:C_0402_1005Metric, F.Cu at (14.3, 73.2)
- added C129: 220p, Capacitor_SMD:C_0402_1005Metric, F.Cu at (14.3, 75.2)
- added C13: 56p, Capacitor_SMD:C_0402_1005Metric, F.Cu at (0.95, 24.4)
- added C130: 1u, Capacitor_SMD:C_0402_1005Metric, F.Cu at (17.2, 61.2)
- added C131: 1n, Capacitor_SMD:C_0402_1005Metric, F.Cu at (17.2, 63.2)
- added C132: DNP, Capacitor_SMD:C_0402_1005Metric, F.Cu at (17.2, 65.2)
- added C133: DNP, Capacitor_SMD:C_0402_1005Metric, F.Cu at (17.2, 67.2)
- added C134: 100n, Capacitor_SMD:C_0402_1005Metric, F.Cu at (17.2, 69.2)
- added C135: 100p, Capacitor_SMD:C_0402_1005Metric, F.Cu at (17.2, 71.2)
- added C136: 100n, Capacitor_SMD:C_0402_1005Metric, F.Cu at (17.2, 73.2)
- added C137: 100n, Capacitor_SMD:C_0402_1005Metric, F.Cu at (17.2, 75.2)
- added C138: 100n, Capacitor_SMD:C_0402_1005Metric, F.Cu at (20.1, 61.2)
- added C139: 100n, Capacitor_SMD:C_0402_1005Metric, F.Cu at (20.1, 63.2)
- added C14: 4u7, Capacitor_SMD:C_0402_1005Metric, F.Cu at (3.87, 0.49)
- added C140: 100n, Capacitor_SMD:C_0402_1005Metric, F.Cu at (20.1, 65.2)
- added C141: 100n, Capacitor_SMD:C_0402_1005Metric, F.Cu at (20.1, 67.2)
- added C142: 100n, Capacitor_SMD:C_0402_1005Metric, F.Cu at (20.1, 69.2)
- added C143: 100u, Capacitor_SMD:CP_Elec_8x10.5, F.Cu at (131.9, 66.8)
- added C144: 100n, Capacitor_SMD:C_0402_1005Metric, F.Cu at (137.0, 62.5)
- added C145: 100n, Capacitor_SMD:C_0402_1005Metric, F.Cu at (138.0, 62.5)
- added C146: 100n, Capacitor_SMD:C_0402_1005Metric, F.Cu at (127.5, 49.8)
- added C147: 100u, Capacitor_SMD:CP_Elec_8x10.5, F.Cu at (155.0, 70.6)
- added C148: 100n, Capacitor_SMD:C_0402_1005Metric, F.Cu at (163.1, 66.5)
- added C149: 100n, Capacitor_SMD:C_0402_1005Metric, F.Cu at (163.1, 68.5)
- added C15: 33n, Capacitor_SMD:C_0402_1005Metric, F.Cu at (3.87, 2.48)
- added C150: 100n, Capacitor_SMD:C_0402_1005Metric, F.Cu at (163.1, 70.5)
- added C151: 100u, Capacitor_SMD:CP_Elec_8x10.5, F.Cu at (177.6, 70.6)
- added C152: 100n, Capacitor_SMD:C_0402_1005Metric, F.Cu at (185.7, 66.5)
- added C153: 100n, Capacitor_SMD:C_0402_1005Metric, F.Cu at (185.7, 68.5)
- added C154: 100n, Capacitor_SMD:C_0402_1005Metric, F.Cu at (185.7, 70.5)
- added C155: 100u, Capacitor_SMD:CP_Elec_8x10.5, F.Cu at (202.0, 69.2)
- added C156: 100n, Capacitor_SMD:C_0402_1005Metric, F.Cu at (196.8, 75.2)
- added C157: 100u, Capacitor_SMD:CP_Elec_8x10.5, F.Cu at (224.6, 69.2)
- added C158: 100n, Capacitor_SMD:C_0402_1005Metric, F.Cu at (219.4, 75.2)
- added C159: 100u, Capacitor_SMD:CP_Elec_8x10.5, F.Cu at (247.2, 69.2)
- added C16: 100n, Capacitor_SMD:C_0402_1005Metric, F.Cu at (3.87, 4.47)
- added C160: 100n, Capacitor_SMD:C_0402_1005Metric, F.Cu at (242.0, 75.2)
- added C17: 1u, Capacitor_SMD:C_0402_1005Metric, F.Cu at (3.87, 6.46)
- added C18: 100n, Capacitor_SMD:C_0402_1005Metric, F.Cu at (3.87, 8.46)
- added C19: 100n, Capacitor_SMD:C_0402_1005Metric, F.Cu at (3.87, 10.4)
- added C20: 100n, Capacitor_SMD:C_0402_1005Metric, F.Cu at (3.87, 12.4)
- added C21: 100n, Capacitor_SMD:C_0402_1005Metric, F.Cu at (3.87, 14.4)
- added C22: 100n, Capacitor_SMD:C_0402_1005Metric, F.Cu at (3.87, 16.4)
- added C23: 100n, Capacitor_SMD:C_0402_1005Metric, F.Cu at (3.87, 18.4)
- added C24: 100n, Capacitor_SMD:C_0402_1005Metric, F.Cu at (3.87, 20.4)
- added C25: 100n, Capacitor_SMD:C_0402_1005Metric, F.Cu at (3.87, 22.4)
- added C26: 100n, Capacitor_SMD:C_0402_1005Metric, F.Cu at (3.87, 24.4)
- added C27: 100n, Capacitor_SMD:C_0402_1005Metric, F.Cu at (6.78, 0.49)
- added C28: 100n, Capacitor_SMD:C_0402_1005Metric, F.Cu at (6.78, 2.48)
- added C29: 100n, Capacitor_SMD:C_0402_1005Metric, F.Cu at (6.78, 4.47)
- added C30: 100n, Capacitor_SMD:C_0402_1005Metric, F.Cu at (6.78, 6.46)
- added C31: 100n, Capacitor_SMD:C_0402_1005Metric, F.Cu at (6.78, 8.46)
- added C32: 100n, Capacitor_SMD:C_0402_1005Metric, F.Cu at (6.78, 10.4)
- added C33: 100n, Capacitor_SMD:C_0402_1005Metric, F.Cu at (6.78, 12.4)
- added C34: 100n, Capacitor_SMD:C_0402_1005Metric, F.Cu at (6.78, 14.4)
- added C35: 100n, Capacitor_SMD:C_0402_1005Metric, F.Cu at (6.78, 16.4)
- added C36: 100n, Capacitor_SMD:C_0402_1005Metric, F.Cu at (6.78, 18.4)
- added C37: 100n, Capacitor_SMD:C_0402_1005Metric, F.Cu at (6.78, 20.4)
- added C38: 100n, Capacitor_SMD:C_0402_1005Metric, F.Cu at (6.78, 22.4)
- added C39: 1u, Capacitor_SMD:C_0402_1005Metric, F.Cu at (6.78, 24.4)
- added C40: 2u2, Capacitor_SMD:C_0402_1005Metric, F.Cu at (9.69, 0.49)
- added C41: TBD, Capacitor_SMD:C_0402_1005Metric, F.Cu at (9.69, 2.48)
- added C42: TBD, Capacitor_SMD:C_0402_1005Metric, F.Cu at (9.69, 4.47)
- added C43: 100n, Capacitor_SMD:C_0402_1005Metric, F.Cu at (9.69, 6.46)
- added C44: 100n, Capacitor_SMD:C_0402_1005Metric, F.Cu at (9.69, 8.46)
- added C45: 1u, Capacitor_SMD:C_0402_1005Metric, F.Cu at (9.69, 10.4)
- added C46: 100n, Capacitor_SMD:C_0402_1005Metric, F.Cu at (9.69, 12.4)
- added C47: 100n, Capacitor_SMD:C_0402_1005Metric, F.Cu at (9.69, 14.4)
- added C48: 100n, Capacitor_SMD:C_0402_1005Metric, F.Cu at (9.69, 16.4)
- added C49: 100n, Capacitor_SMD:C_0402_1005Metric, F.Cu at (9.69, 18.4)
- added C5: 4u7, Capacitor_SMD:C_0402_1005Metric, F.Cu at (0.95, 8.46)
- added C50: 100n, Capacitor_SMD:C_0402_1005Metric, F.Cu at (9.69, 20.4)
- added C51: 100n, Capacitor_SMD:C_0402_1005Metric, F.Cu at (9.69, 22.4)
- added C52: 100n, Capacitor_SMD:C_0402_1005Metric, F.Cu at (9.69, 24.4)
- added C53: 100n, Capacitor_SMD:C_0402_1005Metric, F.Cu at (12.6, 0.49)
- added C54: TBD, Capacitor_SMD:C_0402_1005Metric, F.Cu at (12.6, 2.48)
- added C55: TBD, Capacitor_SMD:C_0402_1005Metric, F.Cu at (12.6, 4.47)
- added C56: 100n, Capacitor_SMD:C_0402_1005Metric, F.Cu at (12.6, 6.46)
- added C57: 100n, Capacitor_SMD:C_0402_1005Metric, F.Cu at (12.6, 8.46)
- added C58: 100n, Capacitor_SMD:C_0402_1005Metric, F.Cu at (12.6, 10.4)
- added C59: 100n, Capacitor_SMD:C_0402_1005Metric, F.Cu at (12.6, 12.4)
- added C6: 4u7, Capacitor_SMD:C_0402_1005Metric, F.Cu at (0.95, 10.4)
- added C60: 100n, Capacitor_SMD:C_0402_1005Metric, F.Cu at (12.6, 14.4)
- added C61: 1u, Capacitor_SMD:C_0402_1005Metric, F.Cu at (12.6, 16.4)
- added C62: 100n, Capacitor_SMD:C_0402_1005Metric, F.Cu at (12.6, 18.4)
- added C63: 1u, Capacitor_SMD:C_0402_1005Metric, F.Cu at (12.6, 20.4)
- added C64: 100n, Capacitor_SMD:C_0402_1005Metric, F.Cu at (12.6, 22.4)
- added C65: 1u, Capacitor_SMD:C_0402_1005Metric, F.Cu at (12.6, 24.4)
- added C66: 1u, Capacitor_SMD:C_0402_1005Metric, F.Cu at (15.5, 0.49)
- added C67: 1u, Capacitor_SMD:C_0402_1005Metric, F.Cu at (15.5, 2.48)
- added C68: 1u, Capacitor_SMD:C_0402_1005Metric, F.Cu at (15.5, 4.47)
- added C69: 100n, Capacitor_SMD:C_0402_1005Metric, F.Cu at (15.5, 6.46)
- added C7: 22u, Capacitor_SMD:C_0402_1005Metric, F.Cu at (0.95, 12.4)
- added C70: 100n, Capacitor_SMD:C_0402_1005Metric, F.Cu at (15.5, 8.46)
- added C71: TBD, Capacitor_SMD:C_0402_1005Metric, F.Cu at (15.5, 10.4)
- added C72: TBD, Capacitor_SMD:C_0402_1005Metric, F.Cu at (15.5, 12.4)
- added C73: 100n, Capacitor_SMD:C_0402_1005Metric, F.Cu at (15.5, 14.4)
- added C74: 47n, Capacitor_SMD:C_0402_1005Metric, F.Cu at (63.5, 71.0)
- added C75: 47n, Capacitor_SMD:C_0402_1005Metric, F.Cu at (63.5, 73.0)
- added C76: 100u, Capacitor_SMD:CP_Elec_8x10.5, F.Cu at (83.3, 75.0)
- added C77: 100u, Capacitor_SMD:CP_Elec_8x10.5, F.Cu at (83.3, 85.0)
- added C78: 1u, Capacitor_SMD:C_0402_1005Metric, F.Cu at (63.5, 75.0)
- added C79: 100n, Capacitor_SMD:C_0402_1005Metric, F.Cu at (63.5, 76.9)
- added C8: 1u, Capacitor_SMD:C_0402_1005Metric, F.Cu at (0.95, 14.4)
- added C80: 100n, Capacitor_SMD:C_0402_1005Metric, F.Cu at (63.5, 78.9)
- added C81: 100n, Capacitor_SMD:C_0402_1005Metric, F.Cu at (63.5, 80.9)
- added C82: 220p, Capacitor_SMD:C_0402_1005Metric, F.Cu at (63.5, 82.9)
- added C83: 220p, Capacitor_SMD:C_0402_1005Metric, F.Cu at (63.5, 84.9)
- added C84: 1u, Capacitor_SMD:C_0402_1005Metric, F.Cu at (66.4, 71.0)
- added C85: 1n, Capacitor_SMD:C_0402_1005Metric, F.Cu at (66.4, 73.0)
- added C86: DNP, Capacitor_SMD:C_0402_1005Metric, F.Cu at (66.4, 75.0)
- added C87: DNP, Capacitor_SMD:C_0402_1005Metric, F.Cu at (66.4, 76.9)
- added C88: 100n, Capacitor_SMD:C_0402_1005Metric, F.Cu at (66.4, 78.9)
- added C89: 100p, Capacitor_SMD:C_0402_1005Metric, F.Cu at (66.4, 80.9)
- added C9: 33n, Capacitor_SMD:C_0402_1005Metric, F.Cu at (0.95, 16.4)
- added C90: 100n, Capacitor_SMD:C_0402_1005Metric, F.Cu at (66.4, 82.9)
- added C91: 100n, Capacitor_SMD:C_0402_1005Metric, F.Cu at (66.4, 84.9)
- added C92: 100n, Capacitor_SMD:C_0402_1005Metric, F.Cu at (69.3, 71.0)
- added C93: 100n, Capacitor_SMD:C_0402_1005Metric, F.Cu at (69.3, 73.0)
- added C94: 100n, Capacitor_SMD:C_0402_1005Metric, F.Cu at (69.3, 75.0)
- added C95: 100n, Capacitor_SMD:C_0402_1005Metric, F.Cu at (69.3, 76.9)
- added C96: 100n, Capacitor_SMD:C_0402_1005Metric, F.Cu at (69.3, 78.9)
- added C97: 47n, Capacitor_SMD:C_0402_1005Metric, F.Cu at (59.0, 17.1)
- added C98: 47n, Capacitor_SMD:C_0402_1005Metric, F.Cu at (59.0, 19.1)
- added C99: 100u, Capacitor_SMD:CP_Elec_8x10.5, F.Cu at (50.9, 4.53)
- added D1: VBUS05B1-SD0, Diode_SMD:D_0603_1608Metric, F.Cu at (1.54, 39.6)
- added D10: VBUS05B1-SD0, Diode_SMD:D_0603_1608Metric, F.Cu at (228.1, 75.5)
- added D11: VBUS05B1-SD0, Diode_SMD:D_0603_1608Metric, F.Cu at (250.7, 75.5)
- added D3: TBD, Diode_SMD:D_0603_1608Metric, F.Cu at (64.1, 97.7)
- added D4: TBD, Diode_SMD:D_0603_1608Metric, F.Cu at (74.2, 23.9)
- added D5: TBD, Diode_SMD:D_0603_1608Metric, F.Cu at (29.4, 68.0)
- added D6: VBUS05B1-SD0, Diode_SMD:D_0603_1608Metric, F.Cu at (137.9, 76.9)
- added D7: VBUS05B1-SD0, Diode_SMD:D_0603_1608Metric, F.Cu at (160.5, 76.9)
- added D8: VBUS05B1-SD0, Diode_SMD:D_0603_1608Metric, F.Cu at (183.1, 76.9)
- added D9: VBUS05B1-SD0, Diode_SMD:D_0603_1608Metric, F.Cu at (205.5, 75.5)
- added FB1: DNP, NetTie:NetTie-2_SMD_Pad0.5mm, F.Cu at (5.08, 39.3)
- added J11: USB_C_Receptacle, Connector_USB:USB3_C_GT-USB-7092A_Right_Angle, B.Cu at (107.5, 45.3)
- added J13: USB_C_Receptacle, Connector_USB:USB3_C_GT-USB-7092A_Right_Angle, B.Cu at (120.9, 45.3)
- added J15: USB3_A, Connector_USB:USB3_A-TH_U231-091N-4BLCC14-S-5, B.Cu at (132.4, 54.5)
- added J16: USB3_A, Connector_USB:USB3_A-TH_U231-091N-4BLCC14-S-5, B.Cu at (159.6, 54.5)
- added J17: USB3_A, Connector_USB:USB3_A-TH_U231-091N-4BLCC14-S-5, B.Cu at (146.0, 54.5)
- added J18: USB3_A, Connector_USB:USB3_A-TH_U231-091N-4BLCC14-S-5, B.Cu at (173.2, 54.5)
- added J19: USB3_A, Connector_USB:USB3_A-TH_U231-091N-4BLCC14-S-5, B.Cu at (186.8, 54.5)
- added J20: USB3_A, Connector_USB:USB3_A-TH_U231-091N-4BLCC14-S-5, B.Cu at (200.4, 54.5)
- added J9: USB_C_Receptacle, Connector_USB:USB3_C_GT-USB-7092A_Right_Angle, B.Cu at (95.5, 45.0)
- added R1: DNP, Resistor_SMD:R_0402_1005Metric, F.Cu at (15.5, 16.4)
- added R10: DNP, Resistor_SMD:R_0402_1005Metric, F.Cu at (18.4, 8.46)
- added R11: 30k9, Resistor_SMD:R_0402_1005Metric, F.Cu at (18.4, 10.4)
- added R12: 10k, Resistor_SMD:R_0402_1005Metric, F.Cu at (18.4, 12.4)
- added R13: 20k, Resistor_SMD:R_0402_1005Metric, F.Cu at (18.4, 14.4)
- added R14: 10k, Resistor_SMD:R_0402_1005Metric, F.Cu at (18.4, 16.4)
- added R15: 10k, Resistor_SMD:R_0402_1005Metric, F.Cu at (18.4, 18.4)
- added R16: 100k, Resistor_SMD:R_0402_1005Metric, F.Cu at (18.4, 20.4)
- added R17: 100k, Resistor_SMD:R_0402_1005Metric, F.Cu at (18.4, 22.4)
- added R18: 10k, Resistor_SMD:R_0402_1005Metric, F.Cu at (18.4, 24.4)
- added R19: 300R, Resistor_SMD:R_0402_1005Metric, F.Cu at (21.3, 0.49)
- added R2: DNP, Resistor_SMD:R_0402_1005Metric, F.Cu at (15.5, 18.4)
- added R20: 1k, Resistor_SMD:R_0402_1005Metric, F.Cu at (21.3, 2.48)
- added R21: 10k, Resistor_SMD:R_0402_1005Metric, F.Cu at (21.3, 4.47)
- added R22: 10k, Resistor_SMD:R_0402_1005Metric, F.Cu at (21.3, 6.46)
- added R23: 10k, Resistor_SMD:R_0402_1005Metric, F.Cu at (21.3, 8.46)
- added R24: 100k, Resistor_SMD:R_0402_1005Metric, F.Cu at (21.3, 10.4)
- added R25: 12k, Resistor_SMD:R_0402_1005Metric, F.Cu at (21.3, 12.4)
- added R26: 12k, Resistor_SMD:R_0402_1005Metric, F.Cu at (21.3, 14.4)
- added R27: 150k, Resistor_SMD:R_0402_1005Metric, F.Cu at (21.3, 16.4)
- added R28: 680R, Resistor_SMD:R_0402_1005Metric, F.Cu at (21.3, 18.4)
- added R29: 5m, Resistor_SMD:R_0402_1005Metric, F.Cu at (69.3, 80.9)
- added R3: 8k66, Resistor_SMD:R_0402_1005Metric, F.Cu at (15.5, 20.4)
- added R30: 10m, Resistor_SMD:R_0402_1005Metric, F.Cu at (69.3, 82.9)
- added R31: 10k, Resistor_SMD:R_0402_1005Metric, F.Cu at (69.3, 84.9)
- added R32: 10k, Resistor_SMD:R_0402_1005Metric, F.Cu at (72.3, 71.0)
- added R33: 10k, Resistor_SMD:R_0402_1005Metric, F.Cu at (72.3, 73.0)
- added R34: 30R1, Resistor_SMD:R_0402_1005Metric, F.Cu at (72.3, 75.0)
- added R35: 30R1, Resistor_SMD:R_0402_1005Metric, F.Cu at (72.3, 76.9)
- added R36: 10k, Resistor_SMD:R_0402_1005Metric, F.Cu at (72.3, 78.9)
- added R37: 10k, Resistor_SMD:R_0402_1005Metric, F.Cu at (72.3, 80.9)
- added R38: 10k, Resistor_SMD:R_0402_1005Metric, F.Cu at (72.3, 82.9)
- added R39: 30R1, Resistor_SMD:R_0402_1005Metric, F.Cu at (72.3, 84.9)
- added R4: 5k, Resistor_SMD:R_0402_1005Metric, F.Cu at (15.5, 22.4)
- added R40: 30R1, Resistor_SMD:R_0402_1005Metric, F.Cu at (75.2, 71.0)
- added R41: DNP, Resistor_SMD:R_0402_1005Metric, F.Cu at (75.2, 73.0)
- added R42: DNP, Resistor_SMD:R_0402_1005Metric, F.Cu at (75.2, 75.0)
- added R43: 50k, Resistor_SMD:R_0402_1005Metric, F.Cu at (75.2, 76.9)
- added R44: 50k, Resistor_SMD:R_0402_1005Metric, F.Cu at (75.2, 78.9)
- added R45: 100k, Resistor_SMD:R_0402_1005Metric, F.Cu at (75.2, 80.9)
- added R46: 300R, Resistor_SMD:R_0402_1005Metric, F.Cu at (75.2, 82.9)
- added R47: 5m, Resistor_SMD:R_0402_1005Metric, F.Cu at (64.8, 27.0)
- added R48: 10m, Resistor_SMD:R_0402_1005Metric, F.Cu at (64.8, 29.0)
- added R49: 10k, Resistor_SMD:R_0402_1005Metric, F.Cu at (64.8, 31.0)
- added R5: 10k, Resistor_SMD:R_0402_1005Metric, F.Cu at (15.5, 24.4)
- added R50: 10k, Resistor_SMD:R_0402_1005Metric, F.Cu at (67.8, 17.1)
- added R51: 10k, Resistor_SMD:R_0402_1005Metric, F.Cu at (67.8, 19.1)
- added R52: 30R1, Resistor_SMD:R_0402_1005Metric, F.Cu at (67.8, 21.1)
- added R53: 30R1, Resistor_SMD:R_0402_1005Metric, F.Cu at (67.8, 23.1)
- added R54: 10k, Resistor_SMD:R_0402_1005Metric, F.Cu at (67.8, 25.1)
- added R55: 10k, Resistor_SMD:R_0402_1005Metric, F.Cu at (67.8, 27.0)
- added R56: 10k, Resistor_SMD:R_0402_1005Metric, F.Cu at (67.8, 29.0)
- added R57: 30R1, Resistor_SMD:R_0402_1005Metric, F.Cu at (67.8, 31.0)
- added R58: 30R1, Resistor_SMD:R_0402_1005Metric, F.Cu at (70.7, 17.1)
- added R59: DNP, Resistor_SMD:R_0402_1005Metric, F.Cu at (70.7, 19.1)
- added R6: 10k, Resistor_SMD:R_0402_1005Metric, F.Cu at (18.4, 0.49)
- added R60: DNP, Resistor_SMD:R_0402_1005Metric, F.Cu at (70.7, 21.1)
- added R61: 50k, Resistor_SMD:R_0402_1005Metric, F.Cu at (70.7, 23.1)
- added R62: 50k, Resistor_SMD:R_0402_1005Metric, F.Cu at (70.7, 25.1)
- added R63: 100k, Resistor_SMD:R_0402_1005Metric, F.Cu at (70.7, 27.0)
- added R64: 300R, Resistor_SMD:R_0402_1005Metric, F.Cu at (70.7, 29.0)
- added R65: 5m, Resistor_SMD:R_0402_1005Metric, F.Cu at (20.1, 71.2)
- added R66: 10m, Resistor_SMD:R_0402_1005Metric, F.Cu at (20.1, 73.2)
- added R67: 10k, Resistor_SMD:R_0402_1005Metric, F.Cu at (20.1, 75.2)
- added R68: 10k, Resistor_SMD:R_0402_1005Metric, F.Cu at (23.0, 61.2)
- added R69: 10k, Resistor_SMD:R_0402_1005Metric, F.Cu at (23.0, 63.2)
- added R7: 20k, Resistor_SMD:R_0402_1005Metric, F.Cu at (18.4, 2.48)
- added R70: 30R1, Resistor_SMD:R_0402_1005Metric, F.Cu at (23.0, 65.2)
- added R71: 30R1, Resistor_SMD:R_0402_1005Metric, F.Cu at (23.0, 67.2)
- added R72: 10k, Resistor_SMD:R_0402_1005Metric, F.Cu at (23.0, 69.2)
- added R73: 10k, Resistor_SMD:R_0402_1005Metric, F.Cu at (23.0, 71.2)
- added R74: 10k, Resistor_SMD:R_0402_1005Metric, F.Cu at (23.0, 73.2)
- added R75: 30R1, Resistor_SMD:R_0402_1005Metric, F.Cu at (23.0, 75.2)
- added R76: 30R1, Resistor_SMD:R_0402_1005Metric, F.Cu at (25.9, 61.2)
- added R77: DNP, Resistor_SMD:R_0402_1005Metric, F.Cu at (25.9, 63.2)
- added R78: DNP, Resistor_SMD:R_0402_1005Metric, F.Cu at (25.9, 65.2)
- added R79: 50k, Resistor_SMD:R_0402_1005Metric, F.Cu at (25.9, 67.2)
- added R8: 10k, Resistor_SMD:R_0402_1005Metric, F.Cu at (18.4, 4.47)
- added R80: 50k, Resistor_SMD:R_0402_1005Metric, F.Cu at (25.9, 69.2)
- added R81: 100k, Resistor_SMD:R_0402_1005Metric, F.Cu at (25.9, 71.2)
- added R82: 300R, Resistor_SMD:R_0402_1005Metric, F.Cu at (25.9, 73.2)
- added R83: 33k2, Resistor_SMD:R_0402_1005Metric, F.Cu at (140.5, 72.5)
- added R84: 300R, Resistor_SMD:R_0402_1005Metric, F.Cu at (127.5, 48.5)
- added R85: 33k2, Resistor_SMD:R_0402_1005Metric, F.Cu at (163.1, 72.5)
- added R86: 300R, Resistor_SMD:R_0402_1005Metric, F.Cu at (163.1, 74.5)
- added R87: 33k2, Resistor_SMD:R_0402_1005Metric, F.Cu at (185.7, 72.5)
- added R88: 300R, Resistor_SMD:R_0402_1005Metric, F.Cu at (185.7, 74.5)
- added R89: 33k2, Resistor_SMD:R_0402_1005Metric, F.Cu at (196.8, 77.2)
- added R9: DNP, Resistor_SMD:R_0402_1005Metric, F.Cu at (18.4, 6.46)
- added R90: 300R, Resistor_SMD:R_0402_1005Metric, F.Cu at (196.8, 79.2)
- added R91: 33k2, Resistor_SMD:R_0402_1005Metric, F.Cu at (219.4, 77.2)
- added R92: 300R, Resistor_SMD:R_0402_1005Metric, F.Cu at (219.4, 79.2)
- added R93: 33k2, Resistor_SMD:R_0402_1005Metric, F.Cu at (242.0, 77.2)
- added R94: 300R, Resistor_SMD:R_0402_1005Metric, F.Cu at (242.0, 79.2)
- added TP1: TestPoint_Small, TestPoint:TestPoint_Pad_D0.5mm, F.Cu at (63.1, 93.4)
- added TP10: TestPoint_Small, TestPoint:TestPoint_Pad_D0.5mm, F.Cu at (45.2, 22.7)
- added TP11: TestPoint_Small, TestPoint:TestPoint_Pad_D0.5mm, F.Cu at (47.3, 20.6)
- added TP12: TestPoint_Small, TestPoint:TestPoint_Pad_D0.5mm, F.Cu at (47.3, 22.7)
- added TP13: TestPoint_Small, TestPoint:TestPoint_Pad_D0.5mm, F.Cu at (49.3, 20.6)
- added TP14: TestPoint_Small, TestPoint:TestPoint_Pad_D0.5mm, F.Cu at (49.3, 22.7)
- added TP15: TestPoint_Small, TestPoint:TestPoint_Pad_D0.5mm, F.Cu at (51.4, 20.6)
- added TP16: TestPoint_Small, TestPoint:TestPoint_Pad_D0.5mm, F.Cu at (51.4, 22.7)
- added TP17: TestPoint_Small, TestPoint:TestPoint_Pad_D0.5mm, F.Cu at (0.53, 64.8)
- added TP18: TestPoint_Small, TestPoint:TestPoint_Pad_D0.5mm, F.Cu at (0.53, 66.8)
- added TP19: TestPoint_Small, TestPoint:TestPoint_Pad_D0.5mm, F.Cu at (2.58, 64.8)
- added TP2: TestPoint_Small, TestPoint:TestPoint_Pad_D0.5mm, F.Cu at (63.1, 95.4)
- added TP20: TestPoint_Small, TestPoint:TestPoint_Pad_D0.5mm, F.Cu at (2.58, 66.8)
- added TP21: TestPoint_Small, TestPoint:TestPoint_Pad_D0.5mm, F.Cu at (4.62, 64.8)
- added TP22: TestPoint_Small, TestPoint:TestPoint_Pad_D0.5mm, F.Cu at (4.62, 66.8)
- added TP23: TestPoint_Small, TestPoint:TestPoint_Pad_D0.5mm, F.Cu at (6.67, 64.8)
- added TP24: TestPoint_Small, TestPoint:TestPoint_Pad_D0.5mm, F.Cu at (6.67, 66.8)
- added TP25: TestPoint_Small, TestPoint:TestPoint_Pad_D0.5mm, F.Cu at (127.2, 70.8)
- added TP26: TestPoint_Small, TestPoint:TestPoint_Pad_D0.5mm, F.Cu at (125.8, 70.8)
- added TP27: TestPoint_Small, TestPoint:TestPoint_Pad_D0.5mm, F.Cu at (154.6, 76.6)
- added TP28: TestPoint_Small, TestPoint:TestPoint_Pad_D0.5mm, F.Cu at (154.6, 78.7)
- added TP29: TestPoint_Small, TestPoint:TestPoint_Pad_D0.5mm, F.Cu at (177.2, 76.6)
- added TP3: TestPoint_Small, TestPoint:TestPoint_Pad_D0.5mm, F.Cu at (65.2, 93.4)
- added TP30: TestPoint_Small, TestPoint:TestPoint_Pad_D0.5mm, F.Cu at (177.2, 78.7)
- added TP4: TestPoint_Small, TestPoint:TestPoint_Pad_D0.5mm, F.Cu at (65.2, 95.4)
- added TP5: TestPoint_Small, TestPoint:TestPoint_Pad_D0.5mm, F.Cu at (67.2, 93.4)
- added TP6: TestPoint_Small, TestPoint:TestPoint_Pad_D0.5mm, F.Cu at (67.2, 95.4)
- added TP7: TestPoint_Small, TestPoint:TestPoint_Pad_D0.5mm, F.Cu at (69.2, 93.4)
- added TP8: TestPoint_Small, TestPoint:TestPoint_Pad_D0.5mm, F.Cu at (69.2, 95.4)
- added TP9: TestPoint_Small, TestPoint:TestPoint_Pad_D0.5mm, F.Cu at (45.2, 20.6)
- added U13: GD25D10CT, Package_SO:SOP-8_3.9x4.9mm_P1.27mm, F.Cu at (3.73, 35.0)
- added U16: ESD122, Package_SON:X2SON-3_L1.0-W0.6-L, F.Cu at (87.0, 97.8)
- added U17: GD25D10CT, Package_SO:SOP-8_3.9x4.9mm_P1.27mm, F.Cu at (66.3, 89.1)
- added U18: ESD122, Package_SON:X2SON-3_L1.0-W0.6-L, F.Cu at (89.1, 97.8)
- added U19: TPD4E02B04, Package_SON:USON-10_2.5x1.0mm_P0.5mm, F.Cu at (72.0, 87.9)
- added U20: HD3SS3212, Package_DFN_QFN:Texas_VQFN-RHL-20, F.Cu at (88.7, 93.3)
- added U21: TPD4E02B04, Package_SON:USON-10_2.5x1.0mm_P0.5mm, F.Cu at (74.8, 87.9)
- added U22: TPS65987DDH, Package_DFN_QFN:TI_VQFN-56, F.Cu at (71.7, 3.83)
- added U23: ACT5101, Package_DFN_QFN:FCQFN-32-3EP_4x4mm_P0.4mm, F.Cu at (52.8, 26.8)
- added U24: ESD122, Package_SON:X2SON-3_L1.0-W0.6-L, F.Cu at (73.1, 21.4)
- added U25: GD25D10CT, Package_SO:SOP-8_3.9x4.9mm_P1.27mm, F.Cu at (70.9, 11.4)
- added U26: ESD122, Package_SON:X2SON-3_L1.0-W0.6-L, F.Cu at (75.2, 21.4)
- added U27: TPD4E02B04, Package_SON:USON-10_2.5x1.0mm_P0.5mm, F.Cu at (73.6, 18.1)
- added U28: HD3SS3212, Package_DFN_QFN:Texas_VQFN-RHL-20, F.Cu at (46.9, 26.9)
- added U29: TPD4E02B04, Package_SON:USON-10_2.5x1.0mm_P0.5mm, F.Cu at (76.4, 18.1)
- added U30: TPS65987DDH, Package_DFN_QFN:TI_VQFN-56, F.Cu at (27.0, 48.0)
- added U31: ACT5101, Package_DFN_QFN:FCQFN-32-3EP_4x4mm_P0.4mm, F.Cu at (8.07, 71.0)
- added U32: ESD122, Package_SON:X2SON-3_L1.0-W0.6-L, F.Cu at (28.4, 65.5)
- added U33: GD25D10CT, Package_SO:SOP-8_3.9x4.9mm_P1.27mm, F.Cu at (26.2, 55.5)
- added U34: ESD122, Package_SON:X2SON-3_L1.0-W0.6-L, F.Cu at (30.5, 65.5)
- added U35: TPD4E02B04, Package_SON:USON-10_2.5x1.0mm_P0.5mm, F.Cu at (28.8, 62.3)
- added U36: HD3SS3212, Package_DFN_QFN:Texas_VQFN-RHL-20, F.Cu at (2.23, 71.1)
- added U37: TPD4E02B04, Package_SON:USON-10_2.5x1.0mm_P0.5mm, F.Cu at (31.7, 62.3)
- added U38: TPS2557, Package_SON:Texas_VSON-8_3x3mm_P0.65_EP2.4x1.65x2.4mm_ThermalVias, F.Cu at (128.2, 73.8)
- added U39: ESD122, Package_SON:X2SON-3_L1.0-W0.6-L, F.Cu at (127.9, 57.1)
- added U40: TPD4E02B04, Package_SON:USON-10_2.5x1.0mm_P0.5mm, F.Cu at (137.2, 54.5)
- added U41: TPS2557, Package_SON:Texas_VSON-8_3x3mm_P0.65_EP2.4x1.65x2.4mm_ThermalVias, F.Cu at (150.9, 77.9)
- added U42: ESD122, Package_SON:X2SON-3_L1.0-W0.6-L, F.Cu at (159.5, 79.4)
- added U43: TPD4E02B04, Package_SON:USON-10_2.5x1.0mm_P0.5mm, F.Cu at (157.0, 77.6)
- added U44: TPS2557, Package_SON:Texas_VSON-8_3x3mm_P0.65_EP2.4x1.65x2.4mm_ThermalVias, F.Cu at (173.5, 77.9)
- added U45: ESD122, Package_SON:X2SON-3_L1.0-W0.6-L, F.Cu at (182.1, 79.4)
- added U46: TPD4E02B04, Package_SON:USON-10_2.5x1.0mm_P0.5mm, F.Cu at (179.6, 77.6)
- added U47: TPS2557, Package_SON:Texas_VSON-8_3x3mm_P0.65_EP2.4x1.65x2.4mm_ThermalVias, F.Cu at (200.9, 76.5)
- added U48: ESD122, Package_SON:X2SON-3_L1.0-W0.6-L, F.Cu at (204.5, 78.0)
- added U49: TPS2557, Package_SON:Texas_VSON-8_3x3mm_P0.65_EP2.4x1.65x2.4mm_ThermalVias, F.Cu at (223.5, 76.5)
- added U50: ESD122, Package_SON:X2SON-3_L1.0-W0.6-L, F.Cu at (227.1, 78.0)
- added U51: TPS2557, Package_SON:Texas_VSON-8_3x3mm_P0.65_EP2.4x1.65x2.4mm_ThermalVias, F.Cu at (246.1, 76.5)
- added U52: ESD122, Package_SON:X2SON-3_L1.0-W0.6-L, F.Cu at (249.7, 78.0)
- added Y1: 25MHz, Crystal:Crystal_SMD_Abracon_ABM8G-4Pin_3.2x2.5mm, F.Cu at (39.6, 21.8)
- added Y2: 24MHz, Crystal:Crystal_SMD_Abracon_ABM8G-4Pin_3.2x2.5mm, F.Cu at (39.6, 26.2)
- added Y3: 25MHz, Crystal:Crystal_SMD_Abracon_ABM8G-4Pin_3.2x2.5mm, F.Cu at (39.6, 30.7)
- C1: value 100n -> 10u; footprint Resistor_SMD:R_0402_1005Metric -> Capacitor_SMD:C_0402_1005Metric
- C2, C3: footprint Resistor_SMD:R_0402_1005Metric -> Capacitor_SMD:C_0402_1005Metric
- C4: value 100n -> 56p; footprint Resistor_SMD:R_0402_1005Metric -> Capacitor_SMD:C_0402_1005Metric
- U10: value TPD4E02B04 -> USB2514B_Bi; footprint Package_SON:USON-10_2.5x1.0mm_P0.5mm -> Package_DFN_QFN:QFN-36-1EP_6x6mm_P0.5mm_EP3.7x3.7mm
- U11: value AP7313-12SAG-7 -> TPS2557; footprint Package_TO_SOT_SMD:SOT-23 -> Package_SON:Texas_VSON-8_3x3mm_P0.65_EP2.4x1.65x2.4mm_ThermalVias
- U12: value TPD4E02B04 -> GL3224; footprint Package_SON:USON-10_2.5x1.0mm_P0.5mm -> Package_DFN_QFN:QFN-48-1EP_7x7mm_P0.5mm_EP5.3x5.3mm_ThermalVias
- U14: value TPD4E02B04 -> TPS65987DDH; footprint Package_SON:USON-10_2.5x1.0mm_P0.5mm -> Package_DFN_QFN:TI_VQFN-56
- U15: value ESD122 -> ACT5101; footprint Package_SON:X2SON-3_L1.0-W0.6-L -> Package_DFN_QFN:FCQFN-32-3EP_4x4mm_P0.4mm
- U2: value TPD4E02B04 -> TPS74801DRCT; footprint Package_SON:USON-10_2.5x1.0mm_P0.5mm -> Package_DFN_QFN:TQFN-20-1EP_5x5mm_P0.65mm_EP3.1x3.1mm_ThermalVias
- U3: value HD3SS3212 -> TPS62932DRLR; footprint Package_DFN_QFN:Texas_VQFN-RHL-20 -> Package_TO_SOT_SMD:SOT-583
- U4: value TPD4E02B04 -> TCA9548AMRGER; footprint Package_SON:USON-10_2.5x1.0mm_P0.5mm -> Package_DFN_QFN:Texas_RGE0024C_EP2.1x2.1mm
- U5: value TPS65987DDH -> USB5807C; footprint Package_DFN_QFN:TI_VQFN-56 -> Package_DFN_QFN:VQFN-100-1EP_12x12mm_P0.4mm_EP8x8mm
- U6: value ACT5101 -> ESD122; footprint Package_DFN_QFN:FCQFN-32-3EP_4x4mm_P0.4mm -> Package_SON:X2SON-3_L1.0-W0.6-L
- U7: value ATtiny3227-M -> TPD4E02B04; footprint Package_DFN_QFN:QFN-24-1EP_4x4mm_P0.5mm_EP2.6x2.6mm -> Package_SON:USON-10_2.5x1.0mm_P0.5mm
- U8: value USB5807C -> ATtiny3227-M; footprint Package_DFN_QFN:VQFN-100-1EP_12x12mm_P0.4mm_EP8x8mm -> Package_DFN_QFN:QFN-24-1EP_4x4mm_P0.5mm_EP2.6x2.6mm
- U9: value ESD122 -> GD25D10CT; footprint Package_SON:X2SON-3_L1.0-W0.6-L -> Package_SO:SOP-8_3.9x4.9mm_P1.27mm
- moved C1 163.8 mm to (0.95, 0.49)
- moved C2 163.8 mm to (0.95, 2.48)
- moved C3 163.8 mm to (0.95, 4.47)
- moved C4 163.8 mm to (0.95, 6.46)
- moved U9 152.4 mm to (3.73, 28.6)
- moved U4 146.4 mm to (11.1, 37.8)
- moved U3 125.4 mm to (32.9, 38.8)
- moved U2 116.6 mm to (38.4, 37.0)
- moved U1 115.1 mm to (32.9, 35.0)
- moved U12 114.4 mm to (12.6, 30.0), turned to 0 degrees
- moved U7 96.4 mm to (18.6, 32.0)
- moved U8 95.2 mm to (17.4, 37.7)
- moved U6 92.1 mm to (21.1, 31.2)
- moved U11 86.0 mm to (19.8, 27.7), turned to 0 degrees
- moved U10 85.7 mm to (26.9, 37.5), turned to 0 degrees
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Connections:
- C1 pad 1: Net-(U12-O3) -> +24V
- C1 pad 2: Net-(J1-TX2+) -> GND
- C2 pad 1: Net-(U12-O4) -> +24V
- C2 pad 2: Net-(J1-TX2-) -> GND
- C3 pad 1: Net-(U2-O4) -> Net-(U1-BST)
- C3 pad 2: Net-(J1-TX1+) -> Net-(U1-SW)
- C4 pad 1: Net-(U2-O3) -> Net-(C4-Pad1)
- C4 pad 2: Net-(J1-TX1-) -> Net-(U1-FB)
- U10 pad 1: Net-(J3-SSTX-) -> /USB2_Port_7/D-
- U10 pad 10: Net-(U10-O1) -> Net-(C45-Pad1)
- U10 pad 2: Net-(J3-SSTX+) -> /USB2_Port_7/D+
- U10 pad 3: GND -> /USB2_Port_8/D-
- U10 pad 4: Net-(J3-SSRX-) -> /USB2_Port_8/D+
- U10 pad 5: Net-(J3-SSRX+) -> Net-(C45-Pad1)
- U10 pad 6: Net-(U10-O4) -> /USB2_Port_9/D-
- U10 pad 7: Net-(U10-O3) -> /USB2_Port_9/D+
- U10 pad 8: GND -> unconnected-(U10-USBDM_DN4/PRT_DIS_M4-Pad8)
- U10 pad 9: Net-(U10-O2) -> unconnected-(U10-USBDP_DN4/PRT_DIS_P4-Pad9)
- U11 pad 1: Net-(U11-VI) -> GND
- U11 pad 2: GND -> +1V5
- U11 pad 3: +1V2 -> +1V5
- U12 pad 1: Net-(U12-I1) -> Net-(J6-DET_B)
- U12 pad 2: Net-(U12-I2) -> unconnected-(U12-MS1_INS/SD1_WP-Pad2)
- U12 pad 4: Net-(U12-I3) -> unconnected-(U12-D--Pad4)
- U12 pad 5: Net-(U12-I4) -> unconnected-(U12-D+-Pad5)
- U12 pad 6: Net-(U12-O4) -> Net-(C65-Pad1)
- U12 pad 7: Net-(U12-O3) -> Net-(U12-TX-)
- U12 pad 8: GND -> Net-(U12-TX+)
- U14 pad 1: Net-(U14-I1) -> PP_HV2
- U14 pad 2: Net-(U14-I2) -> PP_HV2
- U14 pad 3: GND -> Net-(D3-A2)
- U14 pad 4: Net-(U14-I3) -> Net-(D3-A2)
- U14 pad 5: Net-(U14-I4) -> +3V3
- U14 pad 7: Net-(J4-SSTX-) -> GND
- U14 pad 9: Net-(J4-SSRX+) -> unconnected-(U14-LDO_3V3-Pad9)
- U15 pad 2: Net-(J4-D-) -> GND
- U2 pad 1: Net-(U2-I1) -> +1V2
- U2 pad 2: Net-(U2-I2) -> GND
- U2 pad 4: Net-(U2-I3) -> GND
- U2 pad 5: Net-(U2-I4) -> +1V5
- U2 pad 6: Net-(U2-O4) -> +1V5
- U2 pad 7: Net-(U2-O3) -> +1V5
- U2 pad 8: GND -> +1V5
- U3 pad 1: unconnected-(U3-RSVD1-Pad1) -> Net-(U3-RT)
- U3 pad 2: unconnected-(U3-OEn-Pad2) -> Net-(U3-EN)
- U3 pad 3: /RX1- -> +24V
- U3 pad 4: /RX1+ -> GND
- U3 pad 5: unconnected-(U3-GND-Pad5) -> Net-(U3-SW)
- U3 pad 6: unconnected-(U3-VCC-Pad6) -> Net-(U3-BST)
- U3 pad 7: /TX1- -> Net-(U3-SS)
- U3 pad 8: /TX1+ -> Net-(U3-FB)
- U4 pad 1: Net-(J3-D-) -> I2C_DATA1
- U4 pad 10: Net-(U4-O1) -> unconnected-(U4-SD4-Pad10)
- U4 pad 2: Net-(J3-D+) -> I2C_CLK1
- U4 pad 3: GND -> I2C_DATA2
- U4 pad 4: unconnected-(U4-I3-Pad4) -> I2C_CLK2
- U4 pad 5: unconnected-(U4-I4-Pad5) -> I2C_DATA3
- U4 pad 6: unconnected-(U4-O4-Pad6) -> I2C_CLK3
- U4 pad 8: GND -> unconnected-(U4-SC3-Pad8)
- U4 pad 9: Net-(U4-O2) -> GND
- U5 pad 1: PP_HV2 -> Net-(U5-RBIAS)
- U5 pad 10: unconnected-(U5-ADCIN2-Pad10) -> +1V2
- U5 pad 11: PP_HV1 -> /PD_Port_1/SS_RX+
- U5 pad 12: PP_HV1 -> /PD_Port_1/SS_RX-
- U5 pad 13: Net-(U5-VBUS1-Pad13) -> /PD_Port_2/D+
- U5 pad 14: Net-(U5-VBUS1-Pad13) -> /PD_Port_2/D-
- U5 pad 15: GND -> /PD_Port_2/SS_TX+
- U5 pad 16: unconnected-(U5-GPIO0-Pad16) -> /PD_Port_2/SS_TX-
- U5 pad 17: unconnected-(U5-GPIO1-Pad17) -> +1V2
- U5 pad 18: unconnected-(U5-GPIO2-Pad18) -> /PD_Port_2/SS_RX+
- U5 pad 19: GND -> /PD_Port_2/SS_RX-
- U5 pad 2: PP_HV2 -> +3V3
- U5 pad 20: GND -> unconnected-(U5-GPIO12/~{CFG_STRAP}-Pad20)
- U5 pad 23: unconnected-(U5-~{I2C3_IRQ}/IO7-Pad23) -> GND
- U5 pad 24: Net-(U5-C_CC1) -> HUB1_VBUS_DET
- U5 pad 25: unconnected-(U5-PP_CABLE-Pad25) -> HUB0_~{RST}
- U5 pad 26: Net-(U5-C_CC2) -> +1V2
- U5 pad 27: unconnected-(U5-I2C1_SCL-Pad27) -> +3V3
- U5 pad 28: unconnected-(U5-I2C1_SDA-Pad28) -> /PD_Port_3/D+
- U5 pad 29: unconnected-(U5-~{I2C1_IRQ}-Pad29) -> /PD_Port_3/D-
- U5 pad 3: Net-(J1-VBUS-PadA4) -> Net-(U5-XTALI/CLKIN)
- U5 pad 30: unconnected-(U5-GPIO3(HPD)-Pad30) -> /PD_Port_3/SS_TX+
- U5 pad 31: unconnected-(U5-GPIO4-Pad31) -> /PD_Port_3/SS_TX-
- U5 pad 32: unconnected-(U5-I2C2_SCL-Pad32) -> +1V2
- U5 pad 33: unconnected-(U5-I2C2_SDA-Pad33) -> /PD_Port_3/SS_RX+
- U5 pad 34: unconnected-(U5-~{I2C2_IRQ}-Pad34) -> /PD_Port_3/SS_RX-
- U5 pad 35: unconnected-(U5-LDO_1V8-Pad35) -> /USB3_Port_4/D+
- U5 pad 36: unconnected-(U5-SPI_MISO-Pad36) -> /USB3_Port_4/D-
- U5 pad 37: unconnected-(U5-SPI_MOSI-Pad37) -> /USB3_Port_4/SS_TX+
- U5 pad 38: unconnected-(U5-SPI_CLK-Pad38) -> /USB3_Port_4/SS_TX-
- U5 pad 39: unconnected-(U5-~{SPI_CS}-Pad39) -> +1V2
- U5 pad 4: Net-(J1-VBUS-PadA4) -> Net-(U5-XTALO)
- U5 pad 40: unconnected-(U5-GPIO12-Pad40) -> /USB3_Port_4/SS_RX+
- U5 pad 41: unconnected-(U5-GPIO13-Pad41) -> /USB3_Port_4/SS_RX-
- U5 pad 42: unconnected-(U5-GPIO14(PWM)-Pad42) -> +3V3
- U5 pad 43: unconnected-(U5-GPIO15(PWM)-Pad43) -> Net-(U10-USBDP_UP)
- U5 pad 44: unconnected-(U5-HRESET-Pad44) -> Net-(U10-USBDM_UP)
- U5 pad 45: GND -> Net-(U12-TX+)
- U5 pad 46: GND -> Net-(U12-TX-)
- U5 pad 47: GND -> +1V2
- U5 pad 48: unconnected-(U5-GPIO16(PP_EXT1)-Pad48) -> Net-(U5-USB3DN_RXDP5)
- U5 pad 49: unconnected-(U5-GPIO17(PP_EXT2)-Pad49) -> Net-(U5-USB3DN_RXDM5)
- U5 pad 5: unconnected-(U5-VIN_3V3-Pad5) -> +3V3
- U5 pad 51: GND -> VBUS_EN_P6
- U5 pad 52: GND -> PORT_EN_2.0_P5
- U5 pad 53: unconnected-(U5-C_USB_N/IO19-Pad53) -> VBUS_EN_P7
- U5 pad 54: unconnected-(U5-GPIO20-Pad54) -> +3V3
- U5 pad 56: GND -> unconnected-(U5-SPEED_IND3/BC_IND3/GPIO2-Pad56)
- U5 pad 57: GND -> VBUS_EN_P4
- U5 pad 58: GND -> VBUS_EN_P3
- U5 pad 59: GND -> +1V2
- U5 pad 6: unconnected-(U5-ADCIN1-Pad6) -> /PD_Port_1/D+
- U5 pad 7: GND -> /PD_Port_1/D-
- U5 pad 8: GND -> /PD_Port_1/SS_TX+
- U5 pad 9: unconnected-(U5-LDO_3V3-Pad9) -> /PD_Port_1/SS_TX-
- U6 pad 2: GND -> Net-(J3-D-)
- U6 pad 3: Net-(U6-INTBP) -> Net-(J3-D+)
- U7 pad 1: unconnected-(U7-PA2-Pad1) -> Net-(J3-SSTX-)
- U7 pad 10: unconnected-(U7-PB6-Pad10) -> Net-(U5-USB3UP_TXDP)
- U7 pad 2: unconnected-(U7-PA3-Pad2) -> Net-(J3-SSTX+)
- U7 pad 3: Net-(U7-GND-Pad25) -> GND
- U7 pad 4: unconnected-(U7-VCC-Pad4) -> Net-(J3-SSRX-)
- U7 pad 5: unconnected-(U7-PA4-Pad5) -> Net-(J3-SSRX+)
- U7 pad 6: unconnected-(U7-PA5-Pad6) -> Net-(U5-USB3UP_RXDM)
- U7 pad 7: unconnected-(U7-PA6-Pad7) -> Net-(U5-USB3UP_RXDP)
- U7 pad 8: unconnected-(U7-PA7-Pad8) -> GND
- U7 pad 9: unconnected-(U7-PB7-Pad9) -> Net-(U5-USB3UP_TXDM)
- U8 pad 10: +1V2 -> unconnected-(U8-PB6-Pad10)
- U8 pad 11: /RX1+ -> unconnected-(U8-PB5-Pad11)
- U8 pad 12: /RX1- -> unconnected-(U8-PB4-Pad12)
- U8 pad 15: Net-(U14-I4) -> I2C_DATA
- U8 pad 16: Net-(U14-I3) -> I2C_CLK
- U8 pad 17: +1V2 -> unconnected-(U8-PC0-Pad17)
- U8 pad 18: Net-(U14-I2) -> unconnected-(U8-PC1-Pad18)
- U8 pad 19: Net-(U14-I1) -> unconnected-(U8-PC2-Pad19)
- U8 pad 2: +3V3 -> unconnected-(U8-PA3-Pad2)
- U8 pad 23: unconnected-(U8-TESTEN-Pad23) -> Net-(U8-~{RESET}/PA0)
- U8 pad 24: Net-(U8-VBUS_DET) -> unconnected-(U8-PA1-Pad24)
- U8 pad 25: unconnected-(U8-~{RESET}-Pad25) -> GND
- U8 pad 3: Net-(U8-XTALI/CLKIN) -> GND
- U8 pad 4: Net-(U8-XTALO) -> +3V3
- U8 pad 5: +3V3 -> unconnected-(U8-PA4-Pad5)
- U8 pad 6: /D1+ -> unconnected-(U8-PA5-Pad6)
- U8 pad 7: /D1- -> unconnected-(U8-PA6-Pad7)
- U8 pad 8: /TX1+ -> unconnected-(U8-PA7-Pad8)
- U8 pad 9: /TX1- -> unconnected-(U8-PB7-Pad9)
- U9 pad 1: GND -> Net-(U5-SPI_CE_N/GPIO7/~{CFG_NON_REM})
- U9 pad 2: Net-(J1-CC1) -> Net-(U5-SPI_DI/GPIO9/~{CFG_BC_EN})
- U9 pad 3: Net-(J1-CC2) -> +3V3
Routing:
- net /USB3_Port_4/SS_TX+: track 0.00 -> 17.3 mm
- net /USB3_Port_4/SS_TX-: track 0.00 -> 16.6 mm
- net /USB3_Port_4/SS_RX+: track 0.00 -> 14.0 mm
- net /USB3_Port_4/SS_RX-: track 0.00 -> 13.3 mm
- net /USB3_Port_4/D-: track 0.00 -> 6.15 mm
- net /USB3_Port_4/D+: track 0.00 -> 5.59 mm
Other:
- copper layers 2 -> 4

Commit message: idk
Parts:
- removed J11, J13, J9: USB_C_Receptacle, Connector_USB:USB3_C_GT-USB-7092A_Right_Angle
- removed J3: U235-091N-4BLRC16-2, Connector_USB:USB3_B_U235-091N-4BLRC16-2
- removed U1, U3: TPS62932DRLR, Package_TO_SOT_SMD:SOT-583
- removed U11, U38, U41, U44, U47, U49, U51: TPS2557, Package_SON:Texas_VSON-8_3x3mm_P0.65_EP2.4x1.65x2.4mm_ThermalVias
- removed U14, U22, U30: TPS65987DDH, Package_DFN_QFN:TI_VQFN-56
- removed U15, U23, U31: ACT5101, Package_DFN_QFN:FCQFN-32-3EP_4x4mm_P0.4mm
- removed U16, U18, U24, U26, U32, U34, U39, U42, U45, U48, U50, U52, U6: ESD122, Package_SON:X2SON-3_L1.0-W0.6-L
- removed U5: USB5807C, Package_DFN_QFN:VQFN-100-1EP_12x12mm_P0.4mm_EP8x8mm
- J15, J16, J17, J18, J19, J20: moved to F.Cu
- moved D10 215.7 mm to (12.4, 76.4)
- moved C157 210.5 mm to (14.1, 70.1)
- moved C158 210.5 mm to (8.90, 76.1)
- moved R91 210.5 mm to (8.90, 78.1)
- moved R92 210.5 mm to (8.90, 80.1)
- moved D11 208.4 mm to (42.3, 77.6)
- moved C159 203.2 mm to (44.0, 71.2)
- moved C160 203.2 mm to (38.8, 77.3)
- moved R93 203.2 mm to (38.8, 79.3)
- moved R94 203.2 mm to (38.8, 81.2)
- moved D9 139.8 mm to (65.8, 77.6)
- moved C155 134.5 mm to (67.5, 71.2)
- moved C156 134.5 mm to (62.3, 77.3)
- moved R89 134.5 mm to (62.3, 79.3)
- moved R90 134.5 mm to (62.3, 81.2)
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Connections:
- J18 pad 2: Net-(J18-D-) -> /USB2_Port_7/D+
- J18 pad 3: Net-(J18-D+) -> /USB2_Port_7/D-
- J19 pad 2: Net-(J19-D-) -> /USB2_Port_8/D+
- J19 pad 3: Net-(J19-D+) -> /USB2_Port_8/D-
- J20 pad 2: Net-(J20-D-) -> /USB2_Port_9/D+
- J20 pad 3: Net-(J20-D+) -> /USB2_Port_9/D-
Routing:
- net /USB3_Port_4/SS_TX-: track 16.6 -> 24.3 mm
- net /USB3_Port_4/SS_TX+: track 17.3 -> 25.1 mm
- net /USB3_Port_4/D-: track 6.15 -> 0.00 mm
- net /USB3_Port_4/D+: track 5.59 -> 0.00 mm
- net /USB3_Port_4/SS_RX+: track 14.0 -> 17.7 mm
- net /USB3_Port_4/SS_RX-: track 13.3 -> 17.0 mm
