File: hexahub.kicad_sch (KiCad schematic)
At the start: 76 parts, among them J2 24V_in, J3 U235-091N-4BLRC16-2, J7 5V_in, U1 TPS62932DRLR, U10 TPD4E02B04, U11 TPS74801DRCT, U13 GD25D10CT, U2 TPS62932DRLR, U4 TPD4E02B04, U7 ATtiny3227-M, U8 USB5807C, Y1 25MHz

Commit message: more parts
Parts:
- removed U4: TPD4E02B04, Package_SON:USON-10_2.5x1.0mm_P0.5mm, symbol Interface_USB:TPD4E02B04
- added C41, C42, C43, C44, C45, C46, C49, C50: 100n, symbol Device:C_Small
- added C47, C48: TBD, symbol Device:C_Small
- added R14, R21: 10k, symbol Device:R_Small
- added R22: 12k, symbol Device:R_Small
- added U5: ESD122, Package_SON:X2SON-3_L1.0-W0.6-L, symbol Interface_USB:ESD122
- added U9: USB2514B_Bi, Package_DFN_QFN:QFN-36-1EP_6x6mm_P0.5mm_EP3.7x3.7mm, symbol Interface_USB:USB2514B_Bi
- added Y2: 24MHz, symbol Device:Crystal_GND24_Small
- renumbered C21 to C1, C1 to C10, C2 to C11, C3 to C12, C4 to C13, C5 to C14, C6 to C15, C28 to C16, C29 to C17, C30 to C18, C31 to C19, C18 to C2, C26 to C20, C27 to C21, C25 to C22, C24 to C23, C40 to C24, C41 to C25, C42 to C26, C43 to C27, C44 to C28, C39 to C29, C17 to C3, C38 to C30, C37 to C31, C36 to C32, C35 to C33, C33 to C35, C32 to C36, C22 to C37, C23 to C38, C45 to C39, C74 to C4, C53 to C40, C46 to C5, C52 to C6, C20 to C7, C47 to C8, C19 to C9, J2 to J1, J7 to J2, L2 to L1, L3 to L2, L1 to L3, L5 to L4, R15 to R1, R2 to R10, R3 to R11, R4 to R12, R5 to R13, R21 to R15, R22 to R16, R20 to R17, R26 to R18, R27 to R19, R16 to R2, R25 to R20, R17 to R3, R35 to R4, R34 to R5, R18 to R6, R19 to R7, R42 to R8, R1 to R9, U11 to U2, U2 to U3, U8 to U4, U10 to U6, U13 to U8
Connections:
- net +3V3: now also C41.1, C42.1, C43.1, C44.1, C45.1, C46.1, R14.2, R21.2, U9.10 (VDDA33), U9.15 (VDD33), U9.23 (VDD33), U9.27 (VBUS_DET), U9.29 (VDDA33), U9.36 (VDDA33), U9.5 (VDDA33)
- net GND: now also C41.2, C42.2, C43.2, C44.2, C45.2, C46.2, C47.2, C48.2, C49.2, C50.2, R22.1, U5.1 (GND), U9.37 (VSS), Y2.2, Y2.4
- net I2C_CLK: now also U9.24 (SCL/SMBCLK/CFG_SEL0)
- net I2C_DATA: now also U9.22 (SDA/SMBDATA/NON_REM1)
- net at J3.2 (D-): now also U5.2 (IO1)
- net at U4.95 (USB2UP_DM): now also U5.2 (IO1)
- net at J3.3 (D+): now also U5.3 (IO2)
- net at U4.94 (USB2UP_DP): now also U5.3 (IO2)
- net PD_Port_3/D+: now reaches U4.28 (USB2DN_DP3)
- net PD_Port_3/D-: now reaches U4.29 (USB2DN_DM3)
- net PD_Port_3/SS_TX+: now reaches U4.30 (USB3DN_TXDP3)
- net PD_Port_3/SS_TX-: now reaches U4.31 (USB3DN_TXDM3)
- net PD_Port_3/SS_RX+: now reaches U4.33 (USB3DN_RXDP3)
- net PD_Port_3/SS_RX-: now reaches U4.34 (USB3DN_RXDM3)
- net USB3_Port_5/D+: now reaches U4.43 (USB2DN_DP5)
- net USB3_Port_5/D-: now reaches U4.44 (USB2DN_DM5)
- net USB3_Port_5/SS_TX+: now reaches U4.45 (USB3DN_TXDP5)
- net USB3_Port_5/SS_TX-: now reaches U4.46 (USB3DN_TXDM5)
- net USB3_Port_5/SS_RX+: now reaches U4.48 (USB3DN_RXDP5)
- net USB3_Port_5/SS_RX-: now reaches U4.49 (USB3DN_RXDM5)
- net at U4.79 (USB2DN_DP7): now also U9.31 (USBDP_UP)
- net at U4.80 (USB2DN_DM7): now also U9.30 (USBDM_UP)
- net USB3_Port_6/D+: now reaches U4.86 (USB2DN_DP6)
- net USB3_Port_6/D-: now reaches U4.87 (USB2DN_DM6)
- net USB3_Port_6/SS_TX+: now reaches U4.88 (USB3DN_TXDP6)
- net USB3_Port_6/SS_TX-: now reaches U4.89 (USB3DN_TXDM6)
- net USB3_Port_6/SS_RX+: now reaches U4.91 (USB3DN_RXDP6)
- net USB3_Port_6/SS_RX-: now reaches U4.92 (USB3DN_RXDM6)
- net HUB_~{RST} renamed HUB0_~{RST}
- net HUB0_~{RST}: now also R14.1
- net PORT1_D+ renamed PD_Port_1/D+
- net PORT1_D- renamed PD_Port_1/D-
- net PORT1_RX+ renamed PD_Port_1/SS_RX+
- net PORT1_RX- renamed PD_Port_1/SS_RX-
- net PORT1_TX+ renamed PD_Port_1/SS_TX+
- net PORT1_TX- renamed PD_Port_1/SS_TX-
- net PORT2_D+ renamed PD_Port_2/D+
- net PORT2_D- renamed PD_Port_2/D-
- net PORT2_RX+ renamed PD_Port_2/SS_RX+
- net PORT2_RX- renamed PD_Port_2/SS_RX-
- net PORT2_TX+ renamed PD_Port_2/SS_TX+
- net PORT2_TX- renamed PD_Port_2/SS_TX-
- net PORT4_D+ renamed USB3_Port_4/D+
- net PORT4_D- renamed USB3_Port_4/D-
- net PORT4_RX+ renamed USB3_Port_4/SS_RX+
- net PORT4_RX- renamed USB3_Port_4/SS_RX-
- net PORT4_TX+ renamed USB3_Port_4/SS_TX+
- net PORT4_TX- renamed USB3_Port_4/SS_TX-
- new net: C48.1, U9.32 (XTALOUT), Y2.1
- new net: C47.1, U9.33 (XTALIN/CLKIN), Y2.3
- new net: C50.1, U9.14 (CRFILT)
- new net: R22.2, U9.35 (RBIAS)
- new net: C49.1, U9.34 (PLLFILT)
- new net HUB1_~{RST}: R21.1, U9.26 (RESET_N)
- new net USB2_Port_7/D+: U9.2 (USBDP_DN1/PRT_DIS_P1)
- new net USB2_Port_7/D-: U9.1 (USBDM_DN1/PRT_DIS_M1)
- new net USB2_Port_7/VBUS_EN: U9.12 (PRTPWR1/BC_EN1)
- new net USB2_Port_7/VBUS_~{FAULT}: U9.13 (OCS_N1)
- new net USB2_Port_8/D+: U9.4 (USBDP_DN2/PRT_DIS_P2)
- new net USB2_Port_8/D-: U9.3 (USBDM_DN2/PRT_DIS_M2)
- new net USB2_Port_8/VBUS_EN: U9.16 (PRTPWR2/BC_EN2)
- new net USB2_Port_8/VBUS_~{FAULT}: U9.17 (OCS_N2)
- no-connect marks 26 -> 29
Other:
- sheet USB_Port_4 renamed USB3_Port_4
- added sheet PD_Port_3 (pd_port.kicad_sch)
- added sheet USB2_Port_7 (usb2_type_a_port.kicad_sch)
- added sheet USB2_Port_8 (usb2_type_a_port.kicad_sch)
- added sheet USB3_Port_5 (usb3_type_a_port.kicad_sch)
- added sheet USB3_Port_6 (usb3_type_a_port.kicad_sch)
- sheet USB3_Port_4: file usb_port.kicad_sch -> usb3_type_a_port.kicad_sch
- moved on the sheet: C24, C25, C26, C27, C28, C29, C30, C31, C32, C33, C34, C35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

Commit message: work
Parts:
- added C127: 2u2, symbol Device:C_Small
- added C128: 100n, symbol Device:C_Small
- added C129, C130, C131: 1u, symbol Device:C_Small
- added FB1: DNP, symbol Device:FerriteBead_Small
- added J12: HUB0_ISP, symbol Connector_Generic:Conn_01x05
- added J13: HUB1_ISP, symbol Connector_Generic:Conn_01x05
- added R69: 100k, symbol Device:R_Small
- R15: value 43k -> 100k
- R16: value 49k9 -> 100k
- R18, R19: value 12k -> 10k
Connections:
- net +1V2: now also C130.1
- net +3V3: now also C128.1, C131.1, FB1.2; no longer C43.1, C44.1, C45.1, C46.1, U9.10 (VDDA33), U9.15 (VDD33), U9.23 (VDD33), U9.27 (VBUS_DET), U9.29 (VDDA33), U9.36 (VDDA33), U9.5 (VDDA33)
- net GND: now also C127.2, C128.2, C130.2, C131.2, J12.1 (Pin_1), J12.4 (Pin_4), J13.1 (Pin_1), J13.4 (Pin_4), R69.1; no longer C43.2, C44.2, C45.2, C46.2
- net HUB0_~{RST}: now also J12.5 (Pin_5)
- net HUB1_~{RST}: now also J13.5 (Pin_5)
- net I2C_CLK: now also J12.3 (Pin_3), J13.3 (Pin_3)
- net I2C_DATA: now also J12.2 (Pin_2), J13.2 (Pin_2)
- net at D1.2 (A2), J3.1 (VBUS), R15.1: now also C127.1
- net HUB1_VBUS_DET: now reaches R15.2, R16.2, U4.24 (VBUS_DET)
- net HUB1_VBUS_DET: now also U9.27 (VBUS_DET)
- net at U4.65 (SPI_CLK/C_ATTACH3/GPIO4), U8.6 (SCLK): now also R69.2
- new net: C129.1, C43.1, C44.1, C45.1, C46.1, FB1.1, U9.10 (VDDA33), U9.15 (VDD33), U9.23 (VDD33), U9.29 (VDDA33), U9.36 (VDDA33), U9.5 (VDDA33)
- new net: C129.2, C43.2, C44.2, C45.2, C46.2
Other:
- moved on the sheet: C40, C41, C42, C43, C44, C45, C46, C50, R20, R21, U8

Commit message: stuff
Parts:
- added C141: 100n, symbol Device:C_Small
- added R82: 10k, symbol Device:R_Small
- added U47: TCA9548AMRGER, Package_DFN_QFN:Texas_RGE0024C_EP2.1x2.1mm, symbol Interface_Expansion:TCA9548AMRGER
Connections:
- net +3V3: now also C141.1, R82.2, U47.21 (VCC)
- net GND: now also C141.2, U47.18 (A2), U47.22 (A0), U47.23 (A1), U47.9 (GND)
- net I2C_CLK: now also U47.20 (SDA)
- net I2C_DATA: now also U47.19 (SCL)
- new net: R82.1, U47.24 (~{RESET})
- new net I2C_CLK1: U47.2 (SC0)
- new net I2C_CLK2: U47.4 (SC1)
- new net I2C_CLK3: U47.6 (SC2)
- new net I2C_DATA1: U47.1 (SD0)
- new net I2C_DATA2: U47.3 (SD1)
- new net I2C_DATA3: U47.5 (SD2)

Commit message: stuff
Connections:
- net VBUS_EN_P5: now reaches U4.52 (PRT_CTL5/GPIO21)
- net VBUS_EN_P4: now reaches U4.57 (PRT_CTL4/GANG_PWR/GPIO20)
- net VBUS_EN_P3: now reaches U4.58 (PRT_CTL3/GPIO19)
- net VBUS_EN_P2: now reaches U4.62 (PRT_CTL2/GPIO18)
- net VBUS_EN_P1: now reaches U4.70 (PRT_CTL1/GPIO17)
- no-connect marks 29 -> 22
Other:
- sheet PD_Port_1 ports: added VBUS_EN, VBUS_SENSE; removed none
- sheet PD_Port_2 ports: added VBUS_EN, VBUS_SENSE; removed none
- sheet PD_Port_3 ports: added VBUS_EN, VBUS_SENSE; removed none

Commit message: GL3224
Parts:
- added C142: 100n, symbol Device:C_Small
- added D10: D_Small, symbol Device:D_Small
- added J17: Attiny_ISP, symbol Connector_Generic:Conn_01x06
- added R83: 10k, symbol Device:R_Small
- added R84: 1k, symbol Device:R_Small
- added SW1: RST_BTN, symbol Switch:SW_Push
- added SW2: SW_DPDT_x2, symbol Switch:SW_DPDT_x2
Connections:
- net USB3_Port_5/D+ is gone; now on an unnamed net: U4.43 (USB2DN_DP5)
- net USB3_Port_5/D- is gone; now on an unnamed net: U4.44 (USB2DN_DM5)
- net +3V3: now also U7.4 (VCC), C142.1, J17.2 (Pin_2)
- net GND: now also U7.25 (GND), U7.3 (GND), C142.2, J17.1 (Pin_1), SW1.2
- net I2C_CLK: now also R19.1, U7.16 (PB0); no longer R18.1
- net I2C_DATA: now also R18.1, U7.15 (PB1); no longer R19.1
- net VBUS_EN_P6: now also U4.51 (PRT_CTL6/GPIO22)
- net at U7.13 (PB3): now also J17.6 (Pin_6), SW2.6 (C)
- net at U7.14 (PB2): now also J17.5 (Pin_5), SW2.3 (C)
- net at U7.23 (~{RESET}/PA0): now also R83.1, R84.2
- net VBUS_EN_P7: now reaches U4.53 (PRT_CTL7/GPIO23)
- net PORT_EN_3.0_P5: now reaches U4.71 (SPEED_IND6/BC_IND6/GPIO66)
- net at U9.31 (USBDP_UP): no longer U4.79 (USB2DN_DP7)
- net at U9.30 (USBDM_UP): no longer U4.80 (USB2DN_DM7)
- net USB3_Port_7/SS_TX+: now reaches U4.81 (USB3DN_TXDP7)
- net USB3_Port_7/SS_TX-: now reaches U4.82 (USB3DN_TXDM7)
- net USB3_Port_7/SS_RX+: now reaches U4.84 (USB3DN_RXDP7)
- net USB3_Port_7/SS_RX-: now reaches U4.85 (USB3DN_RXDM7)
- net USB3_Port_5/SS_RX+: no longer names the net of U4.48 (USB3DN_RXDP5)
- net USB3_Port_5/SS_RX-: no longer names the net of U4.49 (USB3DN_RXDM5)
- net USB3_Port_5/SS_TX+: no longer names the net of U4.45 (USB3DN_TXDP5)
- net USB3_Port_5/SS_TX-: no longer names the net of U4.46 (USB3DN_TXDM5)
- net VBUS_EN_P5 renamed PORT_EN_2.0_P5
- new net: D10.2 (A), R84.1, SW2.1 (A)
- new net: R83.2, SW1.1
- new net: D10.1 (K), SW2.4 (A)
- new net: J17.4 (Pin_4), SW2.5 (B)
- new net: J17.3 (Pin_3), SW2.2 (B)
- new net USB3_Port_7/D+: U4.79 (USB2DN_DP7)
- new net USB3_Port_7/D-: U4.80 (USB2DN_DM7)
- no-connect marks 22 -> 17
Other:
- removed sheet USB3_Port_5
- added sheet USB3_Port_7 (usb3_type_a_port.kicad_sch)
- sheet PD_Port_1 ports: added none; removed VBUS_SENSE
- sheet PD_Port_2 ports: added none; removed VBUS_SENSE
- sheet PD_Port_3 ports: added none; removed VBUS_SENSE
- note added: "RX TX"
- moved on the sheet: C128, C129, C141, C39, C41, C42, C43, C44, C45, C46, C47, C48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

Commit message: layout
Parts:
- added C58, C59, C60, C62, C64, C69, C70, C73: 100n, Capacitor_SMD:C_0402_1005Metric, symbol Device:C_Small
- added C61, C63, C65, C66, C67, C68: 1u, Capacitor_SMD:C_0402_1005Metric, symbol Device:C_Small
- added C71, C72: TBD, Capacitor_SMD:C_0402_1005Metric, symbol Device:C_Small
- added J6: Micro_SD_Card_Det, symbol Connector:Micro_SD_Card_Det
- added J8: SD_Card, symbol Connector:SD_Card
- added R27: 150k, Resistor_SMD:R_0402_1005Metric, symbol Device:R_Small
- added R28: 680R, Resistor_SMD:R_0402_1005Metric, symbol Device:R_Small
- added U11: TPS2557, Package_SON:Texas_VSON-8_3x3mm_P0.65_EP2.4x1.65x2.4mm_ThermalVias, symbol Power_Management:TPS2557
- added U12: GL3224, Package_DFN_QFN:QFN-48-1EP_7x7mm_P0.5mm_EP5.3x5.3mm_ThermalVias, symbol Interface_USB:GL3224
- added U13: GD25D10CT, Package_SO:SOP-8_3.9x4.9mm_P1.27mm, symbol Memory_Flash:GD25D10CT
- added Y3: 25MHz, Crystal:Crystal_SMD_Abracon_ABM8G-4Pin_3.2x2.5mm, symbol Device:Crystal_GND24_Small
- C1, C10, C13, C14, C15, C4, C5, C6, C7, C9: footprint (none) -> Capacitor_SMD:C_0402_1005Metric
- C11, C12, C2, C3, C46: footprint (none) -> Capacitor_SMD:C_0402_1005Metric; LCSC (none) -> C386075; MPN (none) -> TMK105B7104KVHF
- C16: renamed from C141; footprint (none) -> Capacitor_SMD:C_0402_1005Metric; LCSC (none) -> C386075; MPN (none) -> TMK105B7104KVHF
- C17: renamed from C131; footprint (none) -> Capacitor_SMD:C_0402_1005Metric; LCSC (none) -> C307427; MPN (none) -> CL05B105KQ5NQNC
- C18: renamed from C16; footprint (none) -> Capacitor_SMD:C_0402_1005Metric; LCSC (none) -> C386075; MPN (none) -> TMK105B7104KVHF
- C19: renamed from C17; footprint (none) -> Capacitor_SMD:C_0402_1005Metric; LCSC (none) -> C386075; MPN (none) -> TMK105B7104KVHF
- C20: renamed from C18; footprint (none) -> Capacitor_SMD:C_0402_1005Metric; LCSC (none) -> C386075; MPN (none) -> TMK105B7104KVHF
- C21: renamed from C19; footprint (none) -> Capacitor_SMD:C_0402_1005Metric; LCSC (none) -> C386075; MPN (none) -> TMK105B7104KVHF
- C22: renamed from C20; footprint (none) -> Capacitor_SMD:C_0402_1005Metric; LCSC (none) -> C386075; MPN (none) -> TMK105B7104KVHF
- C23: renamed from C21; footprint (none) -> Capacitor_SMD:C_0402_1005Metric; LCSC (none) -> C386075; MPN (none) -> TMK105B7104KVHF
- C24: renamed from C22; footprint (none) -> Capacitor_SMD:C_0402_1005Metric; LCSC (none) -> C386075; MPN (none) -> TMK105B7104KVHF
- C25: renamed from C23; footprint (none) -> Capacitor_SMD:C_0402_1005Metric; LCSC (none) -> C386075; MPN (none) -> TMK105B7104KVHF
- C26: renamed from C24; footprint (none) -> Capacitor_SMD:C_0402_1005Metric; LCSC (none) -> C386075; MPN (none) -> TMK105B7104KVHF
- C27: renamed from C25; footprint (none) -> Capacitor_SMD:C_0402_1005Metric; LCSC (none) -> C386075; MPN (none) -> TMK105B7104KVHF
- C28: renamed from C26; footprint (none) -> Capacitor_SMD:C_0402_1005Metric; LCSC (none) -> C386075; MPN (none) -> TMK105B7104KVHF
- C29: renamed from C27; footprint (none) -> Capacitor_SMD:C_0402_1005Metric; LCSC (none) -> C386075; MPN (none) -> TMK105B7104KVHF
- C30: renamed from C28; footprint (none) -> Capacitor_SMD:C_0402_1005Metric; LCSC (none) -> C386075; MPN (none) -> TMK105B7104KVHF
- C31: renamed from C29; footprint (none) -> Capacitor_SMD:C_0402_1005Metric; LCSC (none) -> C386075; MPN (none) -> TMK105B7104KVHF
- C32: renamed from C30; footprint (none) -> Capacitor_SMD:C_0402_1005Metric; LCSC (none) -> C386075; MPN (none) -> TMK105B7104KVHF
- C33: renamed from C31; footprint (none) -> Capacitor_SMD:C_0402_1005Metric; LCSC (none) -> C386075; MPN (none) -> TMK105B7104KVHF
- C34: renamed from C32; footprint (none) -> Capacitor_SMD:C_0402_1005Metric; LCSC (none) -> C386075; MPN (none) -> TMK105B7104KVHF
- C35: renamed from C33; footprint (none) -> Capacitor_SMD:C_0402_1005Metric; LCSC (none) -> C386075; MPN (none) -> TMK105B7104KVHF
- C36: renamed from C34; footprint (none) -> Capacitor_SMD:C_0402_1005Metric; LCSC (none) -> C386075; MPN (none) -> TMK105B7104KVHF
- C37: renamed from C35; footprint (none) -> Capacitor_SMD:C_0402_1005Metric; LCSC (none) -> C386075; MPN (none) -> TMK105B7104KVHF
- C38: renamed from C36; footprint (none) -> Capacitor_SMD:C_0402_1005Metric; LCSC (none) -> C386075; MPN (none) -> TMK105B7104KVHF
- C39: renamed from C130; footprint (none) -> Capacitor_SMD:C_0402_1005Metric; LCSC (none) -> C307427; MPN (none) -> CL05B105KQ5NQNC
- C40: renamed from C127; footprint (none) -> Capacitor_SMD:C_0402_1005Metric
- C41: renamed from C37; footprint (none) -> Capacitor_SMD:C_0402_1005Metric
- C42: renamed from C38; footprint (none) -> Capacitor_SMD:C_0402_1005Metric
- C43: renamed from C142; footprint (none) -> Capacitor_SMD:C_0402_1005Metric; LCSC (none) -> C386075; MPN (none) -> TMK105B7104KVHF
- C44: renamed from C39; footprint (none) -> Capacitor_SMD:C_0402_1005Metric; LCSC (none) -> C386075; MPN (none) -> TMK105B7104KVHF
- C45: renamed from C129; footprint (none) -> Capacitor_SMD:C_0402_1005Metric; LCSC (none) -> C307427; MPN (none) -> CL05B105KQ5NQNC
- C47: renamed from C45; footprint (none) -> Capacitor_SMD:C_0402_1005Metric; LCSC (none) -> C386075; MPN (none) -> TMK105B7104KVHF
- C48: renamed from C44; footprint (none) -> Capacitor_SMD:C_0402_1005Metric; LCSC (none) -> C386075; MPN (none) -> TMK105B7104KVHF
- C49: renamed from C43; footprint (none) -> Capacitor_SMD:C_0402_1005Metric; LCSC (none) -> C386075; MPN (none) -> TMK105B7104KVHF
- C50: renamed from C42; footprint (none) -> Capacitor_SMD:C_0402_1005Metric; LCSC (none) -> C386075; MPN (none) -> TMK105B7104KVHF
- C51: renamed from C41; footprint (none) -> Capacitor_SMD:C_0402_1005Metric; LCSC (none) -> C386075; MPN (none) -> TMK105B7104KVHF
- C52: renamed from C128; footprint (none) -> Capacitor_SMD:C_0402_1005Metric; LCSC (none) -> C386075; MPN (none) -> TMK105B7104KVHF
- C53: renamed from C40; footprint (none) -> Capacitor_SMD:C_0402_1005Metric; LCSC (none) -> C386075; MPN (none) -> TMK105B7104KVHF
- C54: renamed from C47; footprint (none) -> Capacitor_SMD:C_0402_1005Metric
- C55: renamed from C48; footprint (none) -> Capacitor_SMD:C_0402_1005Metric
- C56: renamed from C49; footprint (none) -> Capacitor_SMD:C_0402_1005Metric; LCSC (none) -> C386075; MPN (none) -> TMK105B7104KVHF
- C57: renamed from C50; footprint (none) -> Capacitor_SMD:C_0402_1005Metric; LCSC (none) -> C386075; MPN (none) -> TMK105B7104KVHF
- C8: footprint (none) -> Capacitor_SMD:C_0402_1005Metric; LCSC (none) -> C307427; MPN (none) -> CL05B105KQ5NQNC
- D1: LCSC (none) -> C2859524; MPN (none) -> VBUS05B1-SD0-G4-08
- FB1: footprint (none) -> NetTie:NetTie-2_SMD_Pad0.5mm
- R1, R10, R11, R13, R2, R3, R4, R7, R9: footprint (none) -> Resistor_SMD:R_0402_1005Metric
- R12, R5, R6, R8: footprint (none) -> Resistor_SMD:R_0402_1005Metric; LCSC (none) -> C25744; MPN (none) -> 0402WGF1002TCE
- R14: renamed from R82; footprint (none) -> Resistor_SMD:R_0402_1005Metric; LCSC (none) -> C25744; MPN (none) -> 0402WGF1002TCE
- R15: renamed from R14; footprint (none) -> Resistor_SMD:R_0402_1005Metric; LCSC (none) -> C25744; MPN (none) -> 0402WGF1002TCE
- R16: renamed from R15; footprint (none) -> Resistor_SMD:R_0402_1005Metric; LCSC (none) -> C25741; MPN (none) -> 0402WGF1003TCE
- R17: renamed from R16; footprint (none) -> Resistor_SMD:R_0402_1005Metric; LCSC (none) -> C25741; MPN (none) -> 0402WGF1003TCE
- R18: renamed from R83; footprint (none) -> Resistor_SMD:R_0402_1005Metric; LCSC (none) -> C25744; MPN (none) -> 0402WGF1002TCE
- R19: renamed from R17; footprint (none) -> Resistor_SMD:R_0402_1005Metric; LCSC (none) -> C25102; MPN (none) -> 0402WGF3000TCE
- R20: renamed from R84; footprint (none) -> Resistor_SMD:R_0402_1005Metric
- R21: renamed from R18; footprint (none) -> Resistor_SMD:R_0402_1005Metric; LCSC (none) -> C25744; MPN (none) -> 0402WGF1002TCE
- R22: renamed from R19; footprint (none) -> Resistor_SMD:R_0402_1005Metric; LCSC (none) -> C25744; MPN (none) -> 0402WGF1002TCE
- R23: renamed from R21; footprint (none) -> Resistor_SMD:R_0402_1005Metric; LCSC (none) -> C25744; MPN (none) -> 0402WGF1002TCE
- R24: renamed from R69; footprint (none) -> Resistor_SMD:R_0402_1005Metric; LCSC (none) -> C25741; MPN (none) -> 0402WGF1003TCE
- R25: renamed from R20; footprint (none) -> Resistor_SMD:R_0402_1005Metric
- R26: renamed from R22; footprint (none) -> Resistor_SMD:R_0402_1005Metric
- U6: renamed from U5; LCSC (none) -> C544474; MPN (none) -> ESD122DMXR
- U7: renamed from U6; LCSC (none) -> C106794; MPN (none) -> TPD4E02B04DQAR
- U9: renamed from U8; LCSC (none) -> not in stock; MPN (none) -> not in stock
- Y1, Y2: footprint (none) -> Crystal:Crystal_SMD_Abracon_ABM8G-4Pin_3.2x2.5mm
- renumbered D10 to D2, J17 to J4, J12 to J5, J13 to J7, U9 to U10, U47 to U4, U4 to U5, U7 to U8
Connections:
- net +5V is gone; now on net +1V5: J2.2 (Pin_2)
- net +1V5: now also U11.2 (IN), U11.3 (IN)
- net +3V3: now also C73.1, U13.3 (~{WP}), U13.8 (VCC)
- net GND: now also C58.2, C59.2, C60.2, C61.2, C62.2, C63.2, C64.2, C65.2, C66.2, C67.2, C68.2, C71.2, C72.2, C73.2, J6.11 (SHIELD), J6.6 (VSS), J8.12 (SHELL1), J8.13 (SHELL2), J8.3 (VSS), J8.6 (VSS), R27.1, R28.1, U11.1 (GND), U11.9 (GND), U12.12 (GND), U12.3 (GND), U12.49 (GND), U13.4 (GND), Y3.2, Y3.4
- net PORT_EN_3.0_P5: now also U11.4 (EN), U11.8 (~{FAULT})
- net at U5.45 (USB3DN_TXDP5): now also U12.8 (TX+)
- net at U5.46 (USB3DN_TXDM5): now also U12.7 (TX-)
- net at U5.48 (USB3DN_RXDP5): now also C70.1
- net at U5.49 (USB3DN_RXDM5): now also C69.1
- net USB2_Port_9/VBUS_EN: now reaches U10.18 (PRTPWR3/BC_EN3)
- net USB2_Port_9/VBUS_~{FAULT}: now reaches U10.19 (OCS_N3)
- net USB2_Port_9/D-: now reaches U10.6 (USBDM_DN3/PRT_DIS_M3)
- net USB2_Port_9/D+: now reaches U10.7 (USBDP_DN3/PRT_DIS_P3)
- new net: C70.2, U12.11 (RX+)
- new net: C58.1, C59.1, C60.1, C61.1, U12.25 (VDD33), U12.34 (VDD33), U12.44 (VDD33)
- new net: J6.1 (DAT2), U12.42 (S1D2_M1CK)
- new net: J6.2 (DAT3/CD), U12.41 (S1D3_M1D3)
- new net: J6.3 (CMD), U12.40 (S1CM_M1D2)
- new net: J6.4 (VDD), U12.23 (S1M1_VCC)
- new net: J6.5 (CLK), U12.39 (S1CK_M1D0)
- new net: J6.7 (DAT0), U12.38 (S1D0_M1D1)
- new net: J6.8 (DAT1), U12.37 (S1D1_M1BS)
- new net: J6.9 (DET_B), U12.1 (SD1_CDZ)
- new net: C69.2, U12.10 (RX-)
- new net: C63.1, C64.1, U12.9 (AVDD12)
- new net: R27.2, U11.5 (ILIM)
- new net: C71.1, U12.13 (XI), Y3.3
- new net: C72.1, U12.14 (XO), Y3.1
- new net: C65.1, C66.1, U12.15 (AVDD33), U12.6 (AVDD33)
- new net: R28.2, U12.16 (RTERM)
- new net: U12.17 (SPI_MISO), U13.2 (O1/SO)
- new net: U12.18 (SPI_MOSI), U13.5 (SI/IO0)
- new net: U12.19 (SPI_CK), U13.6 (SCLK)
- new net: U12.20 (SPI_CS), U13.1 (~{CS})
- new net: U11.6 (OUT), U11.7 (OUT), U12.22 (VBUS)
- new net: J8.4 (VDD), U12.24 (S2M2_VCC)
- new net: C62.1, U12.26 (VDD12)
- new net: J8.8 (DAT1), U12.27 (D2D1_M2D1)
- new net: J8.7 (DAT0), U12.28 (S2D0_M2D1)
- new net: J8.5 (CLK), U12.29 (S2CK_M2D0)
- new net: J8.2 (CMD), U12.30 (S2CM_M2D2)
- new net: J8.1 (CD/DAT3), U12.31 (S2D3_M2D3)
- new net: J8.9 (DAT2), U12.32 (S2D2_M2CK)
- new net: C68.1, U12.33 (VUHS_2)
- new net: J8.11 (WRITE_PROTECT), U12.35 (MS2_INS/SD2_WP)
- new net: J8.10 (CARD_DETECT), U12.36 (SD2_CDZ)
- new net: C67.1, U12.43 (VUHS_1)
- no-connect marks 17 -> 19
Other:
- added sheet USB2_Port_9 (usb2_type_a_port.kicad_sch)
- moved on the sheet: J5, J7
