File: pd_port.kicad_sch (KiCad schematic)
At the start: 40 parts, among them J1 USB_C_Receptacle, U12 TPD4E02B04, U2 TPD4E02B04, U3 HD3SS3212, U5 TPS65987DDH, U6 ACT5101, U9 ESD122

Commit message: more parts
Parts:
- added C53: 100u, symbol Device:C_Polarized
Connections:
- net AGND: now also C53.2
- net at J1.A4 (VBUS), J1.A9 (VBUS), J1.B4 (VBUS)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: now also C53.1

Commit message: work
Parts:
- added C12 (x2): 220p, symbol Device:C_Small
- added C40: 100n, symbol Device:C_Small
- added J14: Flash_ISP, symbol Connector_Generic:Conn_01x06
- added R14 (x4): 10k, symbol Device:R_Small
- added U8: GD25D10CT, Package_SO:SOP-8_3.9x4.9mm_P1.27mm, symbol Memory_Flash:GD25D10CT
Connections:
- net +3V3: now also C40.1, J14.1 (Pin_1), R14.1, R14.1, U8.3 (~{WP}), U8.8 (VCC)
- net AGND: now also C12.2, C12.2, C40.2, J14.2 (Pin_2), R14.2, R14.2, U8.4 (GND)
- net at U5.10 (ADCIN2): now also R14.1, R14.2
- net at U5.24 (C_CC1), U9.2 (IO1): now also C12.1
- net +5V: now reaches U5.25 (PP_CABLE)
- net at U5.26 (C_CC2), U9.3 (IO2): now also C12.1
- net at U5.36 (SPI_MISO): now also J14.6 (Pin_6), U8.2 (O1/SO)
- net at U5.37 (SPI_MOSI): now also J14.5 (Pin_5), U8.5 (SI/IO0)
- net at U5.38 (SPI_CLK): now also J14.4 (Pin_4), U8.6 (SCLK)
- net at U5.39 (~{SPI_CS}): now also J14.3 (Pin_3), U8.1 (~{CS})
- net at U5.6 (ADCIN1): now also R14.1, R14.2
- no-connect marks 32 -> 26
Other:
- note added: "3V3 GND"
- note added: "I2C Addr (7-bit) 0x23"
- moved on the sheet: C10, C12

Commit message: stuff
Parts:
- added D1: TBD, Diode_SMD:D_0603_1608Metric, symbol Device:D_TVS
- added Q4: Q_PMOS_DGS, symbol Device:Q_PMOS_DGS
- added Q7: Q_NMOS_DGS, symbol Device:Q_NMOS_DGS
- added R14 (x3): 10k, symbol Device:R_Small
- added R14: 90k, symbol Device:R_Small
Connections:
- net AGND: now also D1.1 (A1), Q7.3 (S), R14.2, R14.2
- net PP_HV2: now also Q4.1 (D); no longer R4.2, R6.2
- net at C53.1, J1.A4 (VBUS), J1.A9 (VBUS)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: now also D1.2 (A2)
- new net: Q4.3 (S), R14.1, R14.1, R4.2, R6.2
- new net: Q4.2 (G), Q7.1 (D), R14.2
- new net VBUS_EN: Q7.2 (G), R14.1
- new net VBUS_SENSE: R14.1, R14.2
Other:
- moved on the sheet: C11, C12, C13, C14, C15, C16, C53, C6, C7, C8, C9, L1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

Commit message: stuff
Connections:
- net AGND: now also U3.2 (OEn)
Changed lines of the file:
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@@
   (junction (at 266.7 196.85) (diameter 0) (color 0 0 0 0)
+  )
+  (junction (at 255.27 196.85) (diameter 0) (color 0 0 0 0)
   )
   (junction (at 139.7 137.16) (diameter 0) (color 0 0 0 0)
@@
     (stroke (width 0) (type default))
   )
+  (wire (pts (xy 255.27 162.56) (xy 255.27 196.85))
+    (stroke (width 0) (type default))
+  )
   (wire (pts (xy 167.64 182.88) (xy 167.64 148.59))
     (stroke (width 0) (type default))
@@
     (stroke (width 0) (type default))
   )
-  (wire (pts (xy 251.46 196.85) (xy 266.7 196.85))
+  (wire (pts (xy 255.27 196.85) (xy 266.7 196.85))
+    (stroke (width 0) (type default))
+  )
+  (wire (pts (xy 251.46 196.85) (xy 255.27 196.85))
     (stroke (width 0) (type default))
   )
@@
     (stroke (width 0) (type default))
   )
+  (wire (pts (xy 259.08 162.56) (xy 255.27 162.56))
+    (stroke (width 0) (type default))
+  )

Commit message: GL3224
Parts:
- removed J14: Flash_ISP, symbol Connector_Generic:Conn_01x06
- removed R14: 10k, symbol Device:R_Small
- removed R14: 90k, symbol Device:R_Small
- added J14: Flash_ISP, symbol Connector_Generic:Conn_01x07
- added TP1, TP10, TP13, TP16, TP19, TP28, TP4, TP7: TestPoint_Small, TestPoint:TestPoint_Pad_D0.5mm, symbol Connector:TestPoint_Small
Connections:
- net +3V3: now also J14.1 (Pin_1)
- net AGND: now also J14.2 (Pin_2)
- net PP_HV2: now also TP13.1
- net VBUS_EN: now also TP28.1
- net at C53.1, D1.2 (A2), J1.A4 (VBUS)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: now also TP19.1
- net at Q4.3 (S), R14.1, R4.2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: now also TP10.1
- net at R7.2, R9.2, U6.12 (VINS)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: now also TP16.1
- net at U5.39 (~{SPI_CS}), U8.1 (~{CS}): now also J14.3 (Pin_3)
- net at U5.36 (SPI_MISO), U8.2 (O1/SO): now also J14.6 (Pin_6)
- net at U5.37 (SPI_MOSI), U8.5 (SI/IO0): now also J14.5 (Pin_5)
- net at U5.38 (SPI_CLK), U8.6 (SCLK): now also J14.4 (Pin_4)
- net at U5.32 (I2C2_SCL): now also TP1.1
- net at U5.33 (I2C2_SDA): now also TP4.1
- net at U5.34 (~{I2C2_IRQ}): now also TP7.1
- net at U5.44 (HRESET): now also J14.7 (Pin_7)
- no-connect marks 26 -> 22
Other:
- note removed: "3V3 GND"

Commit message: layout
Parts:
- C76: renamed from C53; footprint (none) -> Capacitor_SMD:CP_Elec_8x10.5; LCSC (none) -> C5162347; MPN (none) -> CS1H101M-CRF10
- C?: renamed from C54; footprint (none) -> Capacitor_SMD:C_0402_1005Metric; LCSC (none) -> C386075; MPN (none) -> TMK105B7104KVHF
- C?: renamed from C10; footprint (none) -> Capacitor_SMD:CP_Elec_8x10.5; LCSC (none) -> C5162347; MPN (none) -> CS1H101M-CRF10
- C?: renamed from C1; footprint Resistor_SMD:R_0402_1005Metric -> Capacitor_SMD:C_0402_1005Metric; LCSC (none) -> C386075; MPN (none) -> TMK105B7104KVHF
- C? (x2): renamed from C12; footprint (none) -> Capacitor_SMD:C_0402_1005Metric; LCSC (none) -> C386075; MPN (none) -> TMK105B7104KVHF
- C?: renamed from C2; footprint Resistor_SMD:R_0402_1005Metric -> Capacitor_SMD:C_0402_1005Metric; LCSC (none) -> C386075; MPN (none) -> TMK105B7104KVHF
- C?: renamed from C4; footprint Resistor_SMD:R_0402_1005Metric -> Capacitor_SMD:C_0402_1005Metric; LCSC (none) -> C386075; MPN (none) -> TMK105B7104KVHF
- C?: renamed from C16; footprint (none) -> Capacitor_SMD:C_0402_1005Metric
- C? (x2): renamed from C12; footprint (none) -> Capacitor_SMD:C_0402_1005Metric; LCSC (none) -> C76960; MPN (none) -> GRM1555C1H220JA01D
- C?: renamed from C6; footprint (none) -> Capacitor_SMD:C_0402_1005Metric; LCSC (none) -> C386075; MPN (none) -> TMK105B7104KVHF
- C?: renamed from C15; footprint (none) -> Capacitor_SMD:C_0402_1005Metric
- C?: renamed from C8; footprint (none) -> Capacitor_SMD:C_0402_1005Metric; LCSC (none) -> C237221; MPN (none) -> 0402B472K500CT
- C?: renamed from C40; footprint (none) -> Capacitor_SMD:C_0402_1005Metric; LCSC (none) -> C386075; MPN (none) -> TMK105B7104KVHF
- C?: renamed from C13; footprint (none) -> Capacitor_SMD:C_0402_1005Metric
- C?: renamed from C9; footprint (none) -> Capacitor_SMD:C_0402_1005Metric; LCSC (none) -> C237221; MPN (none) -> 0402B472K500CT
- C?: renamed from C14; footprint (none) -> Capacitor_SMD:C_0402_1005Metric
- C?: renamed from C5; footprint (none) -> Capacitor_SMD:C_0402_1005Metric; LCSC (none) -> C386075; MPN (none) -> TMK105B7104KVHF
- C?: renamed from C12; footprint (none) -> Capacitor_SMD:C_0402_1005Metric; LCSC (none) -> C307427; MPN (none) -> CL05B105KQ5NQNC
- C?: renamed from C11; footprint (none) -> Capacitor_SMD:C_0402_1005Metric; LCSC (none) -> C386075; MPN (none) -> TMK105B7104KVHF
- C?: renamed from C7; footprint (none) -> Capacitor_SMD:C_0402_1005Metric; LCSC (none) -> C307427; MPN (none) -> CL05B105KQ5NQNC
- C?: renamed from C3; footprint Resistor_SMD:R_0402_1005Metric -> Capacitor_SMD:C_0402_1005Metric; LCSC (none) -> C386075; MPN (none) -> TMK105B7104KVHF
- J?: renamed from J1; footprint Connector_USB:USB_C_Receptacle_Molex-1054500101 -> Connector_USB:USB3_C_GT-USB-7092A_Right_Angle; LCSC (none) -> C3019719; MPN (none) -> GT-USB-7092A
- R?: renamed from R5; footprint (none) -> Resistor_SMD:R_0402_1005Metric; LCSC (none) -> C416516; MPN (none) -> ERJ2RKF30R1X
- R? (x6): renamed from R14; footprint (none) -> Resistor_SMD:R_0402_1005Metric; LCSC (none) -> C25744; MPN (none) -> 0402WGF1002TCE
- R?: renamed from R13; footprint (none) -> Resistor_SMD:R_0402_1005Metric; LCSC (none) -> C166559; MPN (none) -> RTT025002FTH
- R?: renamed from R11; footprint (none) -> Resistor_SMD:R_0402_1005Metric
- R?: renamed from R6; footprint (none) -> Resistor_SMD:R_0402_1005Metric; LCSC (none) -> C416516; MPN (none) -> ERJ2RKF30R1X
- R?: renamed from R4; footprint (none) -> Resistor_SMD:R_0402_1005Metric
- R?: renamed from R8; footprint (none) -> Resistor_SMD:R_0402_1005Metric; LCSC (none) -> C416516; MPN (none) -> ERJ2RKF30R1X
- R?: renamed from R9; footprint (none) -> Resistor_SMD:R_0402_1005Metric
- R?: renamed from R10; footprint (none) -> Resistor_SMD:R_0402_1005Metric; LCSC (none) -> C166559; MPN (none) -> RTT025002FTH
- R?: renamed from R12; footprint (none) -> Resistor_SMD:R_0402_1005Metric
- R?: renamed from R7; footprint (none) -> Resistor_SMD:R_0402_1005Metric; LCSC (none) -> C416516; MPN (none) -> ERJ2RKF30R1X
- R?: renamed from R1; footprint (none) -> Resistor_SMD:R_0402_1005Metric; LCSC (none) -> C25102; MPN (none) -> 0402WGF3000TCE
- R?: renamed from R14; footprint (none) -> Resistor_SMD:R_0402_1005Metric; LCSC (none) -> C25741; MPN (none) -> 0402WGF1003TCE
- U?: renamed from U2; LCSC (none) -> C106794; MPN (none) -> TPD4E02B04DQAR
- U? (x2): renamed from U9; LCSC (none) -> C544474; MPN (none) -> ESD122DMXR
- U?: renamed from U8; LCSC (none) -> not in stock; MPN (none) -> not in stock
- U?: renamed from U3; LCSC (none) -> C544517; MPN (none) -> HD3SS3212IRKSR
- U?: renamed from U6; LCSC (none) -> not in stock; MPN (none) -> not in stock
- U?: renamed from U12; LCSC (none) -> C106794; MPN (none) -> TPD4E02B04DQAR
- U?: renamed from U5; LCSC (none) -> not in stock; MPN (none) -> not in stock
- renumbered D1 to D?, J14 to J10, L1 to L?, Q4 to Q1, Q7 to Q2, TP16 to TP1, TP10 to TP2, TP13 to TP3, TP19 to TP4, TP28 to TP5, TP1 to TP6, TP4 to TP7, TP7 to TP8
