File: usb2_type_a_port.kicad_sch (KiCad schematic)
At the start: 8 parts, among them J10 USB_A, U15 ESD122, U16 TPS2557

Commit message: layout
Parts:
- removed J10: USB_A, Connector_USB:USB_A_TE_292303-7_Horizontal, symbol Connector:USB_A
- added J?: USB3_A, Connector_USB:USB3_A-TH_U231-091N-4BLCC14-S-5, symbol Connector:USB3_A
- C?: renamed from C50; footprint (none) -> Capacitor_SMD:C_0402_1005Metric; LCSC (none) -> C386075; MPN (none) -> TMK105B7104KVHF
- C?: renamed from C51; footprint (none) -> Capacitor_SMD:CP_Elec_8x10.5; LCSC (none) -> C5162347; MPN (none) -> CS1H101M-CRF10
- D?: renamed from D2; LCSC (none) -> C2859524; MPN (none) -> VBUS05B1-SD0-G4-08
- R?: renamed from R23; footprint (none) -> Resistor_SMD:R_0402_1005Metric; LCSC (none) -> C25102; MPN (none) -> 0402WGF3000TCE
- R?: renamed from R24; footprint (none) -> Resistor_SMD:R_0402_1005Metric; LCSC (none) -> C122548; MPN (none) -> 0402WGF3322TCE
- U?: renamed from U16; LCSC (none) -> C130056; MPN (none) -> TPS2557DRBR
- U?: renamed from U15; LCSC (none) -> C544474; MPN (none) -> ESD122DMXR
Connections:
- net GND: now also J?.4 (GND), J?.7 (DRAIN)
- net at C?.2, R?.2: now also J?.10 (SHIELD)
- net at C?.1, D?.2 (A2), U?.6 (OUT)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: now also J?.1 (VBUS)
- new net: J?.2 (D-), U?.2 (IO1)
- new net: J?.3 (D+), U?.3 (IO2)
- no-connect marks 0 -> 4
Other:
- moved on the sheet: C?, R?

Commit message: idk
Connections:
- net D+: now also J?.2 (D-)
- net D-: now also J?.3 (D+)
Other:
- moved on the sheet: U?
Changed lines of the file:
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@@
     (stroke (width 0) (type default))
   )
-  (wire (pts (xy 182.88 57.15) (xy 184.15 57.15))
-    (stroke (width 0) (type default))
-  )
-  (wire (pts (xy 196.85 54.61) (xy 210.82 54.61))
+  (wire (pts (xy 171.45 57.15) (xy 172.72 57.15))
+    (stroke (width 0) (type default))
+  )
+  (wire (pts (xy 185.42 54.61) (xy 210.82 54.61))
     (stroke (width 0) (type default))
   )
@@
     (stroke (width 0) (type default))
   )
-  (wire (pts (xy 182.88 54.61) (xy 184.15 54.61))
-    (stroke (width 0) (type default))
-  )
-  (wire (pts (xy 191.77 60.96) (xy 191.77 62.23))
-    (stroke (width 0) (type default))
-  )
-  (wire (pts (xy 196.85 57.15) (xy 210.82 57.15))
+  (wire (pts (xy 171.45 54.61) (xy 172.72 54.61))
+    (stroke (width 0) (type default))
+  )
+  (wire (pts (xy 180.34 60.96) (xy 180.34 62.23))
+    (stroke (width 0) (type default))
+  )
+  (wire (pts (xy 185.42 57.15) (xy 210.82 57.15))
     (stroke (width 0) (type default))
   )
@@
     (effects (font (size 1.27 1.27)) (justify left bottom))
   )
+  (label "D-" (at 190.5 57.15 0) (fields_autoplaced)
+    (effects (font (size 1.27 1.27)) (justify left bottom))
+  )
+  (label "D+" (at 190.5 54.61 0) (fields_autoplaced)
+    (effects (font (size 1.27 1.27)) (justify left bottom))
+  )
   (hierarchical_label "VBUS_EN" (shape input) (at 99.06 54.61 180) (fields_autoplaced)
     (effects (font (size 1.27 1.27)) (justify right))
   )
-  (hierarchical_label "D-" (shape input) (at 182.88 57.15 180) (fields_autoplaced)
+  (hierarchical_label "D-" (shape input) (at 171.45 57.15 180) (fields_autoplaced)
     (effects (font (size 1.27 1.27)) (justify right))
   )
-  (hierarchical_label "D+" (shape input) (at 182.88 54.61 180) (fields_autoplaced)
+  (hierarchical_label "D+" (shape input) (at 171.45 54.61 180) (fields_autoplaced)
     (effects (font (size 1.27 1.27)) (justify right))
   )
@@
     )
   )
-  (symbol (lib_id "Interface_USB:ESD122") (at 191.77 54.61 0) (unit 1)
+  (symbol (lib_id "Interface_USB:ESD122") (at 180.34 54.61 0) (unit 1)
     (in_bom yes) (on_board yes) (dnp no)
-    (property "Reference" "U?" (at 186.69 50.8 0)
-      (effects (font (size 1.27 1.27)))
-    )
-    (property "Value" "ESD122" (at 194.31 50.8 0)
-      (effects (font (size 1.27 1.27)))
-    )
-    (property "Footprint" "Package_SON:X2SON-3_L1.0-W0.6-L" (at 196.85 59.69 0)
-      (effects (font (size 1.27 1.27)) hide)
-    )
-    (property "Datasheet" "" (at 196.85 59.69 0)
-      (effects (font (size 1.27 1.27)) hide)
-    )
-    (property "LCSC" "C544474" (at 191.77 54.61 0)
-      (effects (font (size 1.27 1.27)) hide)
-    )
-    (property "MPN" "ESD122DMXR" (at 191.77 54.61 0)
+    (property "Reference" "U?" (at 175.26 50.8 0)
+      (effects (font (size 1.27 1.27)))
+    )
+    (property "Value" "ESD122" (at 182.88 50.8 0)
+      (effects (font (size 1.27 1.27)))
+    )
+    (property "Footprint" "Package_SON:X2SON-3_L1.0-W0.6-L" (at 185.42 59.69 0)
+      (effects (font (size 1.27 1.27)) hide)
+    )
+    (property "Datasheet" "" (at 185.42 59.69 0)
+      (effects (font (size 1.27 1.27)) hide)
+    )
+    (property "LCSC" "C544474" (at 180.34 54.61 0)
+      (effects (font (size 1.27 1.27)) hide)
+    )
+    (property "MPN" "ESD122DMXR" (at 180.34 54.61 0)
       (effects (font (size 1.27 1.27)) hide)
     )
@@
     )
   )
-  (symbol (lib_id "power:GND") (at 191.77 60.96 0) (unit 1)
+  (symbol (lib_id "power:GND") (at 180.34 60.96 0) (unit 1)
     (in_bom yes) (on_board yes) (dnp no)
-    (property "Reference" "#PWR?" (at 191.77 67.31 0)
-      (effects (font (size 1.27 1.27)) hide)
-    )
-    (property "Value" "GND" (at 188.1184 62.8331 0)
-      (effects (font (size 1.27 1.27)))
-    )
-    (property "Footprint" "" (at 191.77 60.96 0)
-      (effects (font (size 1.27 1.27)) hide)
-    )
-    (property "Datasheet" "" (at 191.77 60.96 0)
-      (effects (font (size 1.27 1.27)) hide)
-    )
+    (property "Reference" "#PWR?" (at 180.34 67.31 0)
+      (effects (font (size 1.27 1.27)) hide)
+    )
+    (property "Value" "GND" (at 176.6884 62.8331 0)
+      (effects (font (size 1.27 1.27)))
+    )
+    (property "Footprint" "" (at 180.34 60.96 0)
+      (effects (font (size 1.27 1.27)) hide)
+    )
+    (property "Datasheet" "" (at 180.34 60.96 0)
+      (effects (font (size 1.27 1.27)) hide)
+    )
