File: usb3_type_a_port.kicad_sch (KiCad schematic)
At the start: 11 parts, among them J4 USB3_A, U14 TPD4E02B04, U15 ESD122, U16 TPS2557

Commit message: GL3224
Parts:
- added TP19 (x2): TestPoint_Small, TestPoint:TestPoint_Pad_D0.5mm, symbol Connector:TestPoint_Small
Connections:
- net VBUS_EN: now also TP19.1
- net at C51.1, D2.2 (A2), J4.1 (VBUS)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: now also TP19.1
Changed lines of the file:
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@@
   (junction (at 236.22 85.09) (diameter 0) (color 0 0 0 0)
   )
+  (junction (at 66.04 54.61) (diameter 0) (color 0 0 0 0)
+  )
   (junction (at 226.06 87.63) (diameter 0) (color 0 0 0 0)
   )
@@
     (stroke (width 0) (type default))
   )
-  (wire (pts (xy 63.5 48.26) (xy 63.5 49.53))
-    (stroke (width 0) (type default))
-  )
-  (wire (pts (xy 63.5 49.53) (xy 73.66 49.53))
+  (wire (pts (xy 69.85 48.26) (xy 69.85 49.53))
+    (stroke (width 0) (type default))
+  )
+  (wire (pts (xy 69.85 49.53) (xy 73.66 49.53))
     (stroke (width 0) (type default))
   )
@@
     (stroke (width 0) (type default))
   )
+  (wire (pts (xy 66.04 54.61) (xy 69.85 54.61))
+    (stroke (width 0) (type default))
+  )
   (wire (pts (xy 236.22 88.9) (xy 236.22 87.63))
     (stroke (width 0) (type default))
@@
     (stroke (width 0) (type default))
   )
+  (wire (pts (xy 66.04 49.53) (xy 66.04 54.61))
+    (stroke (width 0) (type default))
+  )
   (wire (pts (xy 229.87 85.09) (xy 228.6 85.09))
     (stroke (width 0) (type default))
@@
     (stroke (width 0) (type default))
   )
-  (wire (pts (xy 64.77 54.61) (xy 69.85 54.61))
+  (wire (pts (xy 64.77 54.61) (xy 66.04 54.61))
     (stroke (width 0) (type default))
   )
@@
   )
   (wire (pts (xy 82.55 67.31) (xy 82.55 69.85))
+    (stroke (width 0) (type default))
+  )
+  (wire (pts (xy 109.22 44.45) (xy 109.22 49.53))
     (stroke (width 0) (type default))
   )
@@
     )
   )
+  (symbol (lib_id "Connector:TestPoint_Small") (at 109.22 44.45 0) (mirror y) (unit 1)
+    (in_bom yes) (on_board yes) (dnp no)
+    (property "Reference" "TP19" (at 107.95 44.45 0)
+      (effects (font (size 1.27 1.27)) (justify left))
+    )
+    (property "Value" "TestPoint_Small" (at 107.95 45.72 0)
+      (effects (font (size 1.27 1.27)) (justify left) hide)
+    )
+    (property "Footprint" "TestPoint:TestPoint_Pad_D0.5mm" (at 104.14 44.45 0)
+      (effects (font (size 1.27 1.27)) hide)
+    )
+    (property "Datasheet" "~" (at 104.14 44.45 0)
+      (effects (font (size 1.27 1.27)) hide)
+    )
+    (pin "1")
+    (instances
+      (project "hexahub"
+        (path "/19c5c199-cd5a-414d-8700-31cc57e11bc0/b4f4b8eb-c6ad-4e27-91a3-fdc2b6f37168"
+          (reference "TP19") (unit 1)
+        )
+        (path "/19c5c199-cd5a-414d-8700-31cc57e11bc0/0fb9eab3-3a55-4d77-b670-b2394eec5e18"
+          (reference "TP20") (unit 1)
+        )
+        (path "/19c5c199-cd5a-414d-8700-31cc57e11bc0/20c4c77c-c43a-41b8-abb5-74d66e18cc58"
+          (reference "TP21") (unit 1)
+        )
+        (path "/19c5c199-cd5a-414d-8700-31cc57e11bc0/72f5ea5f-d4da-4b63-9511-f600256a25eb"
+          (reference "TP22") (unit 1)
+        )
+        (path "/19c5c199-cd5a-414d-8700-31cc57e11bc0/db2ec964-eaeb-4a3f-babe-a86e8c4c3412"
+          (reference "TP23") (unit 1)
+        )
+        (path "/19c5c199-cd5a-414d-8700-31cc57e11bc0/d2e100cb-ff48-46fe-85c4-e0b63d9e5596"
+          (reference "TP24") (unit 1)
+        )
+      )
+    )
+  )
   (symbol (lib_id "Device:D_TVS") (at 109.22 54.61 270) (mirror x) (unit 1)
     (in_bom yes) (on_board yes) (dnp no) (fields_autoplaced)
@@
     )
   )
-  (symbol (lib_id "power:+5V") (at 63.5 48.26 0) (unit 1)
+  (symbol (lib_id "power:+5V") (at 69.85 48.26 0) (unit 1)
     (in_bom yes) (on_board yes) (dnp no) (fields_autoplaced)
-    (property "Reference" "#PWR037" (at 63.5 52.07 0)
-      (effects (font (size 1.27 1.27)) hide)
-    )
-    (property "Value" "+5V" (at 63.5 43.18 0)
-      (effects (font (size 1.27 1.27)))
-    )
-    (property "Footprint" "" (at 63.5 48.26 0)
-      (effects (font (size 1.27 1.27)) hide)
-    )
-    (property "Datasheet" "" (at 63.5 48.26 0)
+    (property "Reference" "#PWR037" (at 69.85 52.07 0)
+      (effects (font (size 1.27 1.27)) hide)
+    )
+    (property "Value" "+5V" (at 69.85 43.18 0)
+      (effects (font (size 1.27 1.27)))
+    )
+    (property "Footprint" "" (at 69.85 48.26 0)
+      (effects (font (size 1.27 1.27)) hide)
+    )
+    (property "Datasheet" "" (at 69.85 48.26 0)
       (effects (font (size 1.27 1.27)) hide)
     )
@@
         )
       )
+    )
+  )
+  (symbol (lib_id "Connector:TestPoint_Small") (at 66.04 49.53 0) (mirror y) (unit 1)
+    (in_bom yes) (on_board yes) (dnp no)
+    (property "Reference" "TP19" (at 64.77 49.53 0)
+      (effects (font (size 1.27 1.27)) (justify left))
+    )
+    (property "Value" "TestPoint_Small" (at 64.77 50.8 0)
+      (effects (font (size 1.27 1.27)) (justify left) hide)
+    )
+    (property "Footprint" "TestPoint:TestPoint_Pad_D0.5mm" (at 60.96 49.53 0)
+      (effects (font (size 1.27 1.27)) hide)
+    )
+    (property "Datasheet" "~" (at 60.96 49.53 0)
+      (effects (font (size 1.27 1.27)) hide)
+    )
+    (pin "1")
+    (instances
+      (project "hexahub"
+        (path "/19c5c199-cd5a-414d-8700-31cc57e11bc0/b4f4b8eb-c6ad-4e27-91a3-fdc2b6f37168"
+          (reference "TP19") (unit 1)
+        )
+        (path "/19c5c199-cd5a-414d-8700-31cc57e11bc0/0fb9eab3-3a55-4d77-b670-b2394eec5e18"
+          (reference "TP20") (unit 1)
+        )
+        (path "/19c5c199-cd5a-414d-8700-31cc57e11bc0/20c4c77c-c43a-41b8-abb5-74d66e18cc58"
+          (reference "TP21") (unit 1)
+        )
+        (path "/19c5c199-cd5a-414d-8700-31cc57e11bc0/72f5ea5f-d4da-4b63-9511-f600256a25eb"
+          (reference "TP25") (unit 1)
+        )
+        (path "/19c5c199-cd5a-414d-8700-31cc57e11bc0/db2ec964-eaeb-4a3f-babe-a86e8c4c3412"
+          (reference "TP26") (unit 1)
+        )
+        (path "/19c5c199-cd5a-414d-8700-31cc57e11bc0/d2e100cb-ff48-46fe-85c4-e0b63d9e5596"
+          (reference "TP27") (unit 1)
+        )
+      )

Commit message: layout
Parts:
- C?: renamed from C48; footprint Resistor_SMD:R_0402_1005Metric -> Capacitor_SMD:C_0402_1005Metric; LCSC (none) -> C386075; MPN (none) -> TMK105B7104KVHF
- C?: renamed from C49; footprint Resistor_SMD:R_0402_1005Metric -> Capacitor_SMD:C_0402_1005Metric; LCSC (none) -> C386075; MPN (none) -> TMK105B7104KVHF
- C?: renamed from C50; footprint (none) -> Capacitor_SMD:C_0402_1005Metric; LCSC (none) -> C386075; MPN (none) -> TMK105B7104KVHF
- C?: renamed from C51; footprint (none) -> Capacitor_SMD:CP_Elec_8x10.5; LCSC (none) -> C5162347; MPN (none) -> CS1H101M-CRF10
- D?: renamed from D2; LCSC (none) -> C2859524; MPN (none) -> VBUS05B1-SD0-G4-08
- J?: renamed from J4; footprint (none) -> Connector_USB:USB3_A-TH_U231-091N-4BLCC14-S-5; LCSC (none) -> C388644; MPN (none) -> U231-091N-4BLCC14-S5
- R?: renamed from R23; footprint (none) -> Resistor_SMD:R_0402_1005Metric; LCSC (none) -> C25102; MPN (none) -> 0402WGF3000TCE
- R?: renamed from R24; footprint (none) -> Resistor_SMD:R_0402_1005Metric; LCSC (none) -> C122548; MPN (none) -> 0402WGF3322TCE
- U?: renamed from U14; LCSC (none) -> C106794; MPN (none) -> TPD4E02B04DQAR
- U?: renamed from U15; LCSC (none) -> C544474; MPN (none) -> ESD122DMXR
- U?: renamed from U16; LCSC (none) -> C130056; MPN (none) -> TPS2557DRBR
- renumbered TP19 to TP?
Connections:
- net D+: now also J?.2 (D-), U?.2 (IO1); no longer U?.3 (IO2)
- net D-: now also J?.3 (D+), U?.3 (IO2); no longer U?.2 (IO1)
- net SS_RX+: now also C?.1, C?.2, J?.8 (SSTX-), U?.9 (O2)
- net SS_RX-: now also C?.1, C?.2, J?.9 (SSTX+), U?.10 (O1)
- net SS_TX+: now also J?.5 (SSRX-), U?.6 (O4)
- net SS_TX-: now also J?.6 (SSRX+), U?.7 (O3)
Other:
- note added: "port_swap feature"
- moved on the sheet: C?, D?, J?, R?, TP?, U?
